File: atca-simple-loopback-hub.kicad_sch (KiCad schematic)
At the start: 1 part

Commit message: Project recovered
Other:
- sheet J20: file ATCA_Z2_J20.kicad_sch -> sch/ATCA_Z2_J20.kicad_sch
- sheet J21: file ATCA_Z2_J21.kicad_sch -> sch/ATCA_Z2_J21.kicad_sch
- sheet J22: file ATCA_Z2_J22.kicad_sch -> sch/ATCA_Z2_J22.kicad_sch
- sheet J23: file ATCA_Z2_J23.kicad_sch -> sch/ATCA_Z2_J23.kicad_sch
- sheet J24: file ATCA_Z2_J24.kicad_sch -> sch/ATCA_Z2_J24.kicad_sch
- title: ATCA Template -> ATCA Simple Loopback HUB
Changed lines of the file:
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@@
   (paper "A4")
   (title_block
-    (title "ATCA Template")
-    (date "2023-07-20")
+    (title "ATCA Simple Loopback HUB")
+    (date "2023-09-12")
     (rev "1.0")
     (company "Karlsruhe Institute of Technology (KIT)")
     (comment 1 "Institute for Data Processing and Electronics (IPE)")
     (comment 2 "Luis Ardila")
-    (comment 4 "Licensed under CERN-OHL-S-2.0")
+    (comment 3 "IPE-380-06")
+    (comment 4 "Licensed under CERN-OHL-P-2.0")
   )
-  (bus (pts (xy 127 93.98) (xy 132.08 93.98))
+  (bus (pts (xy 191.77 85.09) (xy 196.85 85.09))
     (stroke (width 0) (type default))
   )
-  (bus (pts (xy 127 91.44) (xy 132.08 91.44))
+  (bus (pts (xy 191.77 82.55) (xy 196.85 82.55))
     (stroke (width 0) (type default))
   )
-  (text "BASE INTERFACE 1-6" (at 163.83 134.62 0)
+  (text "BASE INTERFACE 1-6" (at 228.6 92.71 0)
     (effects (font (size 2.54 2.54) (thickness 0.508) bold) (justify left bottom))
   )
   (text "CLOCK INTERFACE\nUPDATE INTERFACE\nFABRIC INTERFACE 13-15"
-    (at 163.83 44.45 0)
+    (at 228.6 35.56 0)
     (effects (font (size 2.54 2.54) (thickness 0.508) bold) (justify left bottom))
   )
-  (text "BASE INTERFACE 7-16" (at 163.83 157.48 0)
+  (text "BASE INTERFACE 7-16" (at 228.6 106.68 0)
     (effects (font (size 2.54 2.54) (thickness 0.508) bold) (justify left bottom))
   )
-  (text "FABRIC INTERFACE 8-12" (at 163.83 59.69 0)
+  (text "FABRIC INTERFACE 8-12" (at 228.6 49.53 0)
     (effects (font (size 2.54 2.54) (thickness 0.508) bold) (justify left bottom))
   )
-  (text "FABRIC INTERFACE 3-7" (at 163.83 78.74 0)
+  (text "FABRIC INTERFACE 3-7" (at 228.6 68.58 0)
     (effects (font (size 2.54 2.54) (thickness 0.508) bold) (justify left bottom))
   )
-  (text "FABRIC INTERFACE 1-2" (at 163.83 125.73 0)
+  (text "FABRIC INTERFACE 1-2" (at 228.6 83.82 0)
     (effects (font (size 2.54 2.54) (thickness 0.508) bold) (justify left bottom))
   )
-  (hierarchical_label "Z2_ETH1{ETH}" (shape bidirectional) (at 127 93.98 180) (fields_autoplaced)
+  (hierarchical_label "Z2_ETH1{ETH}" (shape bidirectional) (at 191.77 85.09 180) (fields_autoplaced)
     (effects (font (size 1.27 1.27)) (justify right))
   )
-  (hierarchical_label "Z2_ETH0{ETH}" (shape bidirectional) (at 127 91.44 180) (fields_autoplaced)
+  (hierarchical_label "Z2_ETH0{ETH}" (shape bidirectional) (at 191.77 82.55 180) (fields_autoplaced)
     (effects (font (size 1.27 1.27)) (justify right))
   )
@@
     )
     (instances
-      (project "atca_simple_hub"
+      (project "atca-simple-loopback-hub"
         (path "/b1bf14e0-f6d2-45a7-b67f-6500a354b7ad"
           (reference "G1") (unit 1)
@@
     )
   )
-  (sheet (at 223.52 92.71) (size 43.18 22.86)
+  (sheet (at 196.85 118.11) (size 30.48 39.37) (fields_autoplaced)
     (stroke (width 0.1524) (type solid))
     (fill (color 0 0 0 0.0000))
-    (property "Sheetname" "ATCA_Z1" (at 223.52 91.44 0)
+    (property "Sheetname" "ATCA_Z1" (at 196.85 117.3984 0)
       (effects (font (size 1.27 1.27)) (justify left bottom))
     )
-    (property "Sheetfile" "sch/ATCA_Z1.kicad_sch" (at 223.52 116.84 0)
+    (property "Sheetfile" "sch/ATCA_Z1.kicad_sch" (at 196.85 158.0646 0)
       (effects (font (size 1.27 1.27)) (justify left top))
     )
     (instances
-      (project "atca_simple_hub"
+      (project "atca-simple-loopback-hub"
         (path "/b1bf14e0-f6d2-45a7-b67f-6500a354b7ad" (page "3"))
       )
     )
   )
-  (sheet (at 132.08 88.9) (size 30.48 12.7) (fields_autoplaced)
+  (sheet (at 196.85 80.01) (size 30.48 12.7) (fields_autoplaced)
     (stroke (width 0.1524) (type solid))
     (fill (color 0 0 0 0.0000))
-    (property "Sheetname" "J23" (at 132.08 88.1884 0)
+    (property "Sheetname" "J23" (at 196.85 79.2984 0)
       (effects (font (size 1.27 1.27)) (justify left bottom))
     )
-    (property "Sheetfile" "ATCA_Z2_J23.kicad_sch" (at 132.08 102.1846 0)
+    (property "Sheetfile" "sch/ATCA_Z2_J23.kicad_sch" (at 196.85 93.2946 0)
       (effects (font (size 1.27 1.27)) (justify left top))
     )
-    (pin "Z2_ETH0{ETH}" bidirectional (at 132.08 91.44 180)
+    (pin "Z2_ETH0{ETH}" bidirectional (at 196.85 82.55 180)
       (effects (font (size 1.27 1.27)) (justify left))
     )
-    (pin "Z2_ETH1{ETH}" bidirectional (at 132.08 93.98 180)
+    (pin "Z2_ETH1{ETH}" bidirectional (at 196.85 85.09 180)
       (effects (font (size 1.27 1.27)) (justify left))
     )
     (instances
-      (project "atca_simple_hub"
+      (project "atca-simple-loopback-hub"
         (path "/b1bf14e0-f6d2-45a7-b67f-6500a354b7ad" (page "6"))
       )
     )
   )
-  (sheet (at 50.8 113.03) (size 27.94 27.94) (fields_autoplaced)
+  (sheet (at 127 69.85) (size 27.94 27.94) (fields_autoplaced)
     (stroke (width 0.1524) (type solid))
     (fill (color 0 0 0 0.0000))
-    (property "Sheetname" "ETH_Mag_Jacks" (at 50.8 112.3184 0)
+    (property "Sheetname" "ETH_Mag_Jacks" (at 127 69.1384 0)
       (effects (font (size 1.27 1.27)) (justify left bottom))
     )
-    (property "Sheetfile" "sch/ETH_Mag_Jacks.kicad_sch" (at 50.8 141.5546 0)
+    (property "Sheetfile" "sch/ETH_Mag_Jacks.kicad_sch" (at 127 98.3746 0)
       (effects (font (size 1.27 1.27)) (justify left top))
     )
     (instances
-      (project "atca_simple_hub"
+      (project "atca-simple-loopback-hub"
         (path "/b1bf14e0-f6d2-45a7-b67f-6500a354b7ad" (page "9"))
       )
     )
   )
-  (sheet (at 124.46 144.78) (size 30.48 22.86) (fields_autoplaced)
+  (sheet (at 196.85 99.06) (size 30.48 12.7) (fields_autoplaced)
     (stroke (width 0.1524) (type solid))
     (fill (color 0 0 0 0.0000))
-    (property "Sheetname" "J24" (at 124.46 144.0684 0)
+    (property "Sheetname" "J24" (at 196.85 98.3484 0)
       (effects (font (size 1.27 1.27)) (justify left bottom))
     )
-    (property "Sheetfile" "ATCA_Z2_J24.kicad_sch" (at 124.46 168.2246 0)
+    (property "Sheetfile" "sch/ATCA_Z2_J24.kicad_sch" (at 196.85 112.3446 0)
       (effects (font (size 1.27 1.27)) (justify left top))
     )
     (instances
-      (project "atca_simple_hub"
+      (project "atca-simple-loopback-hub"
         (path "/b1bf14e0-f6d2-45a7-b67f-6500a354b7ad" (page "8"))
       )
     )
   )
-  (sheet (at 132.08 69.85) (size 30.48 12.7) (fields_autoplaced)
+  (sheet (at 196.85 60.96) (size 30.48 12.7) (fields_autoplaced)
     (stroke (width 0.1524) (type solid))
     (fill (color 0 0 0 0.0000))
-    (property "Sheetname" "J22" (at 132.08 69.1384 0)
+    (property "Sheetname" "J22" (at 196.85 60.2484 0)
       (effects (font (size 1.27 1.27)) (justify left bottom))
     )
-    (property "Sheetfile" "ATCA_Z2_J22.kicad_sch" (at 132.08 83.1346 0)
+    (property "Sheetfile" "sch/ATCA_Z2_J22.kicad_sch" (at 196.85 74.2446 0)
       (effects (font (size 1.27 1.27)) (justify left top))
     )
     (instances
-      (project "atca_simple_hub"
+      (project "atca-simple-loopback-hub"
         (path "/b1bf14e0-f6d2-45a7-b67f-6500a354b7ad" (page "7"))
       )
     )
   )
-  (sheet (at 132.08 50.8) (size 30.48 12.7) (fields_autoplaced)
+  (sheet (at 196.85 41.91) (size 30.48 12.7) (fields_autoplaced)
     (stroke (width 0.1524) (type solid))
     (fill (color 0 0 0 0.0000))
-    (property "Sheetname" "J21" (at 132.08 50.0884 0)
+    (property "Sheetname" "J21" (at 196.85 41.1984 0)
       (effects (font (size 1.27 1.27)) (justify left bottom))
     )
-    (property "Sheetfile" "ATCA_Z2_J21.kicad_sch" (at 132.08 64.0846 0)
+    (property "Sheetfile" "sch/ATCA_Z2_J21.kicad_sch" (at 196.85 55.1946 0)
       (effects (font (size 1.27 1.27)) (justify left top))
     )
     (instances
-      (project "atca_simple_hub"
+      (project "atca-simple-loopback-hub"
         (path "/b1bf14e0-f6d2-45a7-b67f-6500a354b7ad" (page "9"))
       )
     )
   )
-  (sheet (at 132.08 31.75) (size 30.48 12.7) (fields_autoplaced)
+  (sheet (at 196.85 22.86) (size 30.48 12.7) (fields_autoplaced)
     (stroke (width 0.1524) (type solid))
     (fill (color 0 0 0 0.0000))
-    (property "Sheetname" "J20" (at 132.08 31.0384 0)
+    (property "Sheetname" "J20" (at 196.85 22.1484 0)
       (effects (font (size 1.27 1.27)) (justify left bottom))
     )
-    (property "Sheetfile" "ATCA_Z2_J20.kicad_sch" (at 132.08 45.0346 0)
+    (property "Sheetfile" "sch/ATCA_Z2_J20.kicad_sch" (at 196.85 36.1446 0)
       (effects (font (size 1.27 1.27)) (justify left top))
     )
     (instances
-      (project "atca_simple_hub"
+      (project "atca-simple-loopback-hub"
         (path "/b1bf14e0-f6d2-45a7-b67f-6500a354b7ad" (page "5"))
       )
     )
   )
-  (sheet (at 190.5 17.78) (size 24.13 10.16) (fields_autoplaced)
+  (sheet (at 149.86 182.88) (size 24.13 10.16) (fields_autoplaced)
     (stroke (width 0.1524) (type solid))
     (fill (color 0 0 0 0.0000))
-    (property "Sheetname" "mech" (at 190.5 17.0684 0)
+    (property "Sheetname" "mech" (at 149.86 182.1684 0)
       (effects (font (size 1.27 1.27)) (justify left bottom))
     )
-    (property "Sheetfile" "sch/mech.kicad_sch" (at 190.5 28.5246 0)
+    (property "Sheetfile" "sch/mech.kicad_sch" (at 149.86 193.6246 0)
       (effects (font (size 1.27 1.27)) (justify left top))
     )
     (instances
-      (project "atca_simple_hub"
+      (project "atca-simple-loopback-hub"
         (path "/b1bf14e0-f6d2-45a7-b67f-6500a354b7ad" (page "2"))
       )

Commit message: BI and FI
Other:
- sheet ETH_Mag_Jacks ports: added Z2_BI1{ETH}, Z2_BI2{ETH}, Z2_BI3{ETH}, Z2_BI4{ETH}, Z2_BI5{ETH}, Z2_BI6{ETH}, Z2_BI7{ETH}, Z2_BI8{ETH}; removed none
- sheet J23 ports: added Z2_BI1{ETH}, Z2_BI2{ETH}, Z2_BI3{ETH}, Z2_BI4{ETH}, Z2_BI5{ETH}, Z2_BI6{ETH}; removed Z2_ETH0{ETH}, Z2_ETH1{ETH}
- sheet J24 ports: added Z2_BI7{ETH}, Z2_BI8{ETH}; removed none
Changed lines of the file:
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@@
     (comment 4 "Licensed under CERN-OHL-P-2.0")
   )
-  (bus (pts (xy 191.77 85.09) (xy 196.85 85.09))
+  (bus (pts (xy 157.48 97.79) (xy 196.85 97.79))
     (stroke (width 0) (type default))
   )
-  (bus (pts (xy 191.77 82.55) (xy 196.85 82.55))
+  (bus (pts (xy 157.48 100.33) (xy 196.85 100.33))
     (stroke (width 0) (type default))
   )
-  (text "BASE INTERFACE 1-6" (at 228.6 92.71 0)
+  (bus (pts (xy 179.07 121.92) (xy 196.85 121.92))
+    (stroke (width 0) (type default))
+  )
+  (bus (pts (xy 157.48 102.87) (xy 196.85 102.87))
+    (stroke (width 0) (type default))
+  )
+  (bus (pts (xy 157.48 105.41) (xy 196.85 105.41))
+    (stroke (width 0) (type default))
+  )
+  (bus (pts (xy 179.07 113.03) (xy 179.07 121.92))
+    (stroke (width 0) (type default))
+  )
+  (bus (pts (xy 176.53 115.57) (xy 176.53 124.46))
+    (stroke (width 0) (type default))
+  )
+  (bus (pts (xy 157.48 107.95) (xy 196.85 107.95))
+    (stroke (width 0) (type default))
+  )
+  (bus (pts (xy 157.48 113.03) (xy 179.07 113.03))
+    (stroke (width 0) (type default))
+  )
+  (bus (pts (xy 157.48 115.57) (xy 176.53 115.57))
+    (stroke (width 0) (type default))
+  )
+  (bus (pts (xy 176.53 124.46) (xy 196.85 124.46))
+    (stroke (width 0) (type default))
+  )
+  (bus (pts (xy 157.48 110.49) (xy 196.85 110.49))
+    (stroke (width 0) (type default))
+  )
+  (text "BASE INTERFACE 1-6" (at 228.6 105.41 0)
     (effects (font (size 2.54 2.54) (thickness 0.508) bold) (justify left bottom))
   )
@@
     (effects (font (size 2.54 2.54) (thickness 0.508) bold) (justify left bottom))
   )
-  (text "BASE INTERFACE 7-16" (at 228.6 106.68 0)
+  (text "BASE INTERFACE 7-16" (at 228.6 124.46 0)
     (effects (font (size 2.54 2.54) (thickness 0.508) bold) (justify left bottom))
   )
@@
     (effects (font (size 2.54 2.54) (thickness 0.508) bold) (justify left bottom))
   )
-  (text "FABRIC INTERFACE 1-2" (at 228.6 83.82 0)
+  (text "FABRIC INTERFACE 1-2" (at 228.6 91.44 0)
     (effects (font (size 2.54 2.54) (thickness 0.508) bold) (justify left bottom))
-  )
-  (hierarchical_label "Z2_ETH1{ETH}" (shape bidirectional) (at 191.77 85.09 180) (fields_autoplaced)
-    (effects (font (size 1.27 1.27)) (justify right))
-  )
-  (hierarchical_label "Z2_ETH0{ETH}" (shape bidirectional) (at 191.77 82.55 180) (fields_autoplaced)
-    (effects (font (size 1.27 1.27)) (justify right))
   )
   (symbol (lib_id "project:KIT_LOGO") (at 267.97 173.99 0) (unit 1)
@@
     )
   )
-  (sheet (at 196.85 118.11) (size 30.48 39.37) (fields_autoplaced)
+  (sheet (at 196.85 133.35) (size 30.48 29.21) (fields_autoplaced)
     (stroke (width 0.1524) (type solid))
     (fill (color 0 0 0 0.0000))
-    (property "Sheetname" "ATCA_Z1" (at 196.85 117.3984 0)
+    (property "Sheetname" "ATCA_Z1" (at 196.85 132.6384 0)
       (effects (font (size 1.27 1.27)) (justify left bottom))
     )
-    (property "Sheetfile" "sch/ATCA_Z1.kicad_sch" (at 196.85 158.0646 0)
+    (property "Sheetfile" "sch/ATCA_Z1.kicad_sch" (at 196.85 163.1446 0)
       (effects (font (size 1.27 1.27)) (justify left top))
     )
@@
     )
   )
-  (sheet (at 196.85 80.01) (size 30.48 12.7) (fields_autoplaced)
+  (sheet (at 196.85 85.09) (size 30.48 27.94) (fields_autoplaced)
     (stroke (width 0.1524) (type solid))
     (fill (color 0 0 0 0.0000))
-    (property "Sheetname" "J23" (at 196.85 79.2984 0)
+    (property "Sheetname" "J23" (at 196.85 84.3784 0)
       (effects (font (size 1.27 1.27)) (justify left bottom))
     )
-    (property "Sheetfile" "sch/ATCA_Z2_J23.kicad_sch" (at 196.85 93.2946 0)
+    (property "Sheetfile" "sch/ATCA_Z2_J23.kicad_sch" (at 196.85 113.6146 0)
       (effects (font (size 1.27 1.27)) (justify left top))
     )
-    (pin "Z2_ETH0{ETH}" bidirectional (at 196.85 82.55 180)
+    (pin "Z2_BI6{ETH}" input (at 196.85 110.49 180)
       (effects (font (size 1.27 1.27)) (justify left))
     )
-    (pin "Z2_ETH1{ETH}" bidirectional (at 196.85 85.09 180)
+    (pin "Z2_BI5{ETH}" input (at 196.85 107.95 180)
+      (effects (font (size 1.27 1.27)) (justify left))
+    )
+    (pin "Z2_BI4{ETH}" input (at 196.85 105.41 180)
+      (effects (font (size 1.27 1.27)) (justify left))
+    )
+    (pin "Z2_BI3{ETH}" input (at 196.85 102.87 180)
+      (effects (font (size 1.27 1.27)) (justify left))
+    )
+    (pin "Z2_BI2{ETH}" bidirectional (at 196.85 100.33 180)
+      (effects (font (size 1.27 1.27)) (justify left))
+    )
+    (pin "Z2_BI1{ETH}" bidirectional (at 196.85 97.79 180)
       (effects (font (size 1.27 1.27)) (justify left))
     )
@@
     )
   )
-  (sheet (at 127 69.85) (size 27.94 27.94) (fields_autoplaced)
+  (sheet (at 129.54 95.25) (size 27.94 22.86) (fields_autoplaced)
     (stroke (width 0.1524) (type solid))
     (fill (color 0 0 0 0.0000))
-    (property "Sheetname" "ETH_Mag_Jacks" (at 127 69.1384 0)
+    (property "Sheetname" "ETH_Mag_Jacks" (at 129.54 94.5384 0)
       (effects (font (size 1.27 1.27)) (justify left bottom))
     )
-    (property "Sheetfile" "sch/ETH_Mag_Jacks.kicad_sch" (at 127 98.3746 0)
+    (property "Sheetfile" "sch/ETH_Mag_Jacks.kicad_sch" (at 129.54 118.6946 0)
       (effects (font (size 1.27 1.27)) (justify left top))
+    )
+    (pin "Z2_BI3{ETH}" input (at 157.48 102.87 0)
+      (effects (font (size 1.27 1.27)) (justify right))
+    )
+    (pin "Z2_BI4{ETH}" input (at 157.48 105.41 0)
+      (effects (font (size 1.27 1.27)) (justify right))
+    )
+    (pin "Z2_BI2{ETH}" bidirectional (at 157.48 100.33 0)
+      (effects (font (size 1.27 1.27)) (justify right))
+    )
+    (pin "Z2_BI1{ETH}" bidirectional (at 157.48 97.79 0)
+      (effects (font (size 1.27 1.27)) (justify right))
+    )
+    (pin "Z2_BI6{ETH}" input (at 157.48 110.49 0)
+      (effects (font (size 1.27 1.27)) (justify right))
+    )
+    (pin "Z2_BI5{ETH}" input (at 157.48 107.95 0)
+      (effects (font (size 1.27 1.27)) (justify right))
+    )
+    (pin "Z2_BI7{ETH}" input (at 157.48 113.03 0)
+      (effects (font (size 1.27 1.27)) (justify right))
+    )
+    (pin "Z2_BI8{ETH}" input (at 157.48 115.57 0)
+      (effects (font (size 1.27 1.27)) (justify right))
     )
     (instances
@@
     )
   )
-  (sheet (at 196.85 99.06) (size 30.48 12.7) (fields_autoplaced)
+  (sheet (at 196.85 119.38) (size 30.48 7.62) (fields_autoplaced)
     (stroke (width 0.1524) (type solid))
     (fill (color 0 0 0 0.0000))
-    (property "Sheetname" "J24" (at 196.85 98.3484 0)
+    (property "Sheetname" "J24" (at 196.85 118.6684 0)
       (effects (font (size 1.27 1.27)) (justify left bottom))
     )
-    (property "Sheetfile" "sch/ATCA_Z2_J24.kicad_sch" (at 196.85 112.3446 0)
+    (property "Sheetfile" "sch/ATCA_Z2_J24.kicad_sch" (at 196.85 127.5846 0)
       (effects (font (size 1.27 1.27)) (justify left top))
     )
+    (pin "Z2_BI8{ETH}" input (at 196.85 124.46 180)
+      (effects (font (size 1.27 1.27)) (justify left))
+    )
+    (pin "Z2_BI7{ETH}" input (at 196.85 121.92 180)
+      (effects (font (size 1.27 1.27)) (justify left))
+    )
     (instances
