File: atca-simple-loopback-hub.kicad_pcb (KiCad board)
At the start: 12 copper layers, 99.9 x 193 mm, 48 parts, among them J1 0826-1X4T-HS-F, J10 Conn_Coaxial, J11 Conn_Coaxial, J12 Conn_Coaxial, J13 Conn_Coaxial, J14 Conn_01x02_Pin, J15 Conn_01x02_Pin, J16 TE 2007262-1, J2 0826-1X4T-HS-F, J20 TE_64690XX-1_J20, J21 TE_64690XX-1_J21, J22 TE_64690XX-1_J22, J23 TE_64690XX-1_J23, J24 TE_64690XX-1_J24, J3 ESD_strip_bottom, J4 Conn_Coaxial, J5 Conn_Coaxial, J6 SFP+, J7 SFP+, J8 Conn_Coaxial, J9 Conn_Coaxial, K2 Key_K1_K2_TE_1-1469373-1, P10 1766500-1, U1 Si5395, U2 Si5395, U3 Pico

Commit message: sch work
Parts:
- removed R7, R8: 4.7k, Resistor_SMD:R_0402_1005Metric
- added C10: 0.1uF, Capacitor_SMD:C_0402_1005Metric, F.Cu at (296.2, 229.8)
- added C11: 0.1uF, Capacitor_SMD:C_0402_1005Metric, F.Cu at (297.2, 229.8)
- added C12: 0.1uF, Capacitor_SMD:C_0402_1005Metric, F.Cu at (295.2, 229.8)
- added C13: 0.1uF, Capacitor_SMD:C_0402_1005Metric, F.Cu at (306.2, 237.8)
- added C14: 0.1uF, Capacitor_SMD:C_0402_1005Metric, F.Cu at (303.5, 247.8)
- added C15: 0.1uF, Capacitor_SMD:C_0402_1005Metric, F.Cu at (297.5, 234.2)
- added C16: 0.1uF, Capacitor_SMD:C_0402_1005Metric, F.Cu at (292.2, 244.2)
- added C17: 0.1uF, Capacitor_SMD:C_0402_1005Metric, F.Cu at (306.2, 245.0)
- added C18: 0.1uF, Capacitor_SMD:C_0402_1005Metric, F.Cu at (306.2, 243.2)
- added C19: 0.1uF, Capacitor_SMD:C_0402_1005Metric, F.Cu at (306.2, 239.5)
- added C20: 0.1uF, Capacitor_SMD:C_0402_1005Metric, F.Cu at (306.2, 241.2)
- added C203: 22uF, Capacitor_SMD:C_1210_3225Metric, F.Cu at (527.2, 160.6)
- added C205: 22uF, Capacitor_SMD:C_1210_3225Metric, B.Cu at (527.2, 160.6)
- added C206: 22uF, Capacitor_SMD:C_1210_3225Metric, B.Cu at (533.7, 160.6)
- added C208: 22uF, Capacitor_SMD:C_1210_3225Metric, F.Cu at (533.7, 160.6)
- added C21: 0.1uF, Capacitor_SMD:C_0402_1005Metric, F.Cu at (298.0, 247.7)
- added C22: 0.1uF, Capacitor_SMD:C_0402_1005Metric, F.Cu at (300.0, 247.8)
- added C23: 0.1uF, Capacitor_SMD:C_0402_1005Metric, F.Cu at (301.7, 247.8)
- added C24: 0.1uF, Capacitor_SMD:C_0402_1005Metric, F.Cu at (301.5, 234.2)
- added C25: 0.1uF, Capacitor_SMD:C_0402_1005Metric, F.Cu at (303.2, 234.2)
- added C26: 0.1uF, Capacitor_SMD:C_0402_1005Metric, F.Cu at (293.2, 254.8)
- added C27: 0.1uF, Capacitor_SMD:C_0402_1005Metric, F.Cu at (296.2, 254.8)
- added C28: 0.1uF, Capacitor_SMD:C_0402_1005Metric, F.Cu at (294.2, 254.8)
- added C29: 0.1uF, Capacitor_SMD:C_0402_1005Metric, F.Cu at (292.2, 254.8)
- added C30: 0.1uF, Capacitor_SMD:C_0402_1005Metric, F.Cu at (297.2, 254.8)
- added C31: 0.1uF, Capacitor_SMD:C_0402_1005Metric, F.Cu at (295.2, 254.8)
- added C32: 0.1uF, Capacitor_SMD:C_0402_1005Metric, F.Cu at (306.2, 262.8)
- added C33: 0.1uF, Capacitor_SMD:C_0402_1005Metric, F.Cu at (303.5, 272.8)
- added C34: 0.1uF, Capacitor_SMD:C_0402_1005Metric, F.Cu at (297.5, 259.2)
- added C35: 0.1uF, Capacitor_SMD:C_0402_1005Metric, F.Cu at (292.2, 269.2)
- added C36: 0.1uF, Capacitor_SMD:C_0402_1005Metric, F.Cu at (301.7, 272.8)
- added C37: 0.1uF, Capacitor_SMD:C_0402_1005Metric, F.Cu at (306.2, 268.2)
- added C38: 0.1uF, Capacitor_SMD:C_0402_1005Metric, F.Cu at (306.2, 266.2)
- added C39: 0.1uF, Capacitor_SMD:C_0402_1005Metric, F.Cu at (306.2, 264.5)
- added C40: 0.1uF, Capacitor_SMD:C_0402_1005Metric, F.Cu at (303.2, 259.2)
- added C401: 10uF, Capacitor_SMD:C_0603_1608Metric, F.Cu at (531.2, 163.8)
- added C401, C63: 10uF, Capacitor_SMD:C_0603_1608Metric, F.Cu at (526.0, 181.9)
- added C402, C64: 10uF, Capacitor_SMD:C_0805_2012Metric, F.Cu at (525.2, 184.7)
- added C402: 10uF, Capacitor_SMD:C_0805_2012Metric, F.Cu at (530.4, 166.6)
- added C403, C65: 10uF, Capacitor_SMD:C_0805_2012Metric, F.Cu at (525.2, 186.7)
- added C403: 10uF, Capacitor_SMD:C_0805_2012Metric, F.Cu at (530.4, 168.6)
- added C404: 1uF, Capacitor_SMD:C_0402_1005Metric, B.Cu at (519.2, 186.6)
- added C404: 1uF, Capacitor_SMD:C_0402_1005Metric, B.Cu at (524.2, 168.5)
- added C405: 0.1uF, Capacitor_SMD:C_0402_1005Metric, B.Cu at (522.9, 164.7)
- added C405: 0.1uF, Capacitor_SMD:C_0402_1005Metric, B.Cu at (517.9, 182.8)
- added C406: 47uF, Capacitor_SMD:C_0805_2012Metric, B.Cu at (513.0, 182.2)
- added C406: 47uF, Capacitor_SMD:C_0805_2012Metric, B.Cu at (517.9, 164.1)
- added C407: 47uF, Capacitor_SMD:C_0805_2012Metric, F.Cu at (517.9, 164.1)
- added C408: C, Capacitor_SMD:C_0402_1005Metric, F.Cu at (516.4, 166.8)
- added C41: 0.1uF, Capacitor_SMD:C_0402_1005Metric, F.Cu at (301.5, 259.2)
- added C42: 0.1uF, Capacitor_SMD:C_0402_1005Metric, F.Cu at (306.2, 270.0)
- added C43: 0.1uF, Capacitor_SMD:C_0402_1005Metric, F.Cu at (300.0, 272.8)
- added C44: 0.1uF, Capacitor_SMD:C_0402_1005Metric, F.Cu at (298.0, 272.7)
- added C45: 0.1uF, Capacitor_SMD:C_0402_1005Metric, F.Cu at (478.7, 178.8)
- added C46: 0.1uF, Capacitor_SMD:C_0402_1005Metric, F.Cu at (478.7, 180.7)
- added C47: 0.1uF, Capacitor_SMD:C_0402_1005Metric, F.Cu at (478.7, 182.7)
- added C48: 0.1uF, Capacitor_SMD:C_0402_1005Metric, F.Cu at (478.7, 184.7)
- added C49: 4700pF, project:VISAY_CAP_MY5UCR, F.Cu at (439.2, 148.4)
- added C50: 47uF, project:CHEMI-KE0, F.Cu at (410.5, 292.0)
- added C52: 4700pF, project:VISAY_CAP_MY5UCR, F.Cu at (439.2, 158.7)
- added C53: 4700pF, project:VISAY_CAP_MY5UCR, F.Cu at (439.2, 169.1)
- added C54: 4700pF, project:VISAY_CAP_MY5UCR, F.Cu at (439.2, 179.4)
- added C55: 47uF, project:CHEMI-KE0, F.Cu at (431.5, 261.5)
- added C56: 4700pF, project:VISAY_CAP_MY5UCR, F.Cu at (431.5, 273.5)
- added C57: 2.2uF, Capacitor_SMD:C_1206_3216Metric, F.Cu at (332.7, 339.8)
- added C58: 2.2uF, Capacitor_SMD:C_1206_3216Metric, F.Cu at (460.2, 323.4)
- added C59: 2.2uF, Capacitor_SMD:C_1206_3216Metric, F.Cu at (336.5, 339.8)
- added C60: 2.2uF, Capacitor_SMD:C_1206_3216Metric, F.Cu at (460.2, 330.1)
- added C62: 4700pF, project:VISAY_CAP_MY5UCR, F.Cu at (439.2, 200.0)
- added C66: 1uF, Capacitor_SMD:C_0402_1005Metric, F.Cu at (521.7, 189.9)
- added C67: 0.1uF, Capacitor_SMD:C_0402_1005Metric, F.Cu at (517.0, 179.9)
- added C68: 47uF, Capacitor_SMD:C_0805_2012Metric, F.Cu at (479.5, 168.0)
- added C69: 47uF, Capacitor_SMD:C_0805_2012Metric, F.Cu at (479.5, 171.1)
- added C7: 0.1uF, Capacitor_SMD:C_0402_1005Metric, F.Cu at (293.2, 229.8)
- added C70: 10uF, Capacitor_SMD:C_0603_1608Metric, F.Cu at (486.7, 153.8)
- added C71: 10uF, Capacitor_SMD:C_0805_2012Metric, F.Cu at (479.5, 144.8)
- added C72: 10uF, Capacitor_SMD:C_0805_2012Metric, F.Cu at (479.5, 147.8)
- added C73: 1uF, Capacitor_SMD:C_0402_1005Metric, F.Cu at (490.1, 153.5)
- added C74: 0.1uF, Capacitor_SMD:C_0402_1005Metric, F.Cu at (490.1, 155.5)
- added C75: 47uF, Capacitor_SMD:C_0805_2012Metric, F.Cu at (479.5, 150.8)
- added C76: 47uF, Capacitor_SMD:C_0805_2012Metric, F.Cu at (479.5, 153.8)
- added C8: 0.1uF, Capacitor_SMD:C_0402_1005Metric, F.Cu at (294.2, 229.8)
- added C9: 0.1uF, Capacitor_SMD:C_0402_1005Metric, F.Cu at (292.2, 229.8)
- added D1: BAS21, Package_TO_SOT_SMD:SOT-23, F.Cu at (438.7, 130.1)
- added D2: BAS21, Package_TO_SOT_SMD:SOT-23, F.Cu at (465.5, 325.0)
- added D3: BAS21, Package_TO_SOT_SMD:SOT-23, F.Cu at (465.5, 329.5)
- added D4: SMBJ5347B-TP, project:SMBJ5347B-TP_DO-214AA, F.Cu at (437.5, 214.0)
- added FB1: FerriteBead, Inductor_SMD:L_0603_1608Metric, F.Cu at (291.7, 245.5)
- added FB2: FerriteBead, Inductor_SMD:L_0603_1608Metric, F.Cu at (291.7, 270.5)
- added L1, L401: BLM18SG121TZ1D, Inductor_SMD:L_0603_1608Metric, F.Cu at (524.0, 181.9)
- added L2: BLM18SG121TZ1D, Inductor_SMD:L_0603_1608Metric, F.Cu at (486.7, 156.3)
- added L401: BLM18SG121TZ1D, Inductor_SMD:L_0603_1608Metric, F.Cu at (529.2, 163.8)
- added NT401: Net-Tie_2, KIT_NetTie:NetTie-2_SMD_Pad0.3mm, B.Cu at (524.8, 165.3)
- added NT401: Net-Tie_2, KIT_NetTie:NetTie-2_SMD_Pad0.3mm, B.Cu at (519.8, 183.4)
- added Q1: IRF3710Z, project:D2PAK_TO-263AB_INF, F.Cu at (449.5, 319.2)
- added Q2: IRF3710Z, project:D2PAK_TO-263AB_INF, F.Cu at (437.5, 319.2)
- added Q3: IRF3710Z, project:D2PAK_TO-263AB_INF, F.Cu at (412.5, 314.8)
- added Q4: IRF3710Z, project:D2PAK_TO-263AB_INF, F.Cu at (424.5, 314.8)
- added R13: 50, Resistor_SMD:R_0402_1005Metric, F.Cu at (293.7, 231.8)
- added R14: 50, Resistor_SMD:R_0402_1005Metric, F.Cu at (292.7, 231.8)
- added R15: 50, Resistor_SMD:R_0402_1005Metric, F.Cu at (296.7, 231.8)
- added R16: 50, Resistor_SMD:R_0402_1005Metric, F.Cu at (295.7, 231.8)
- added R17: 4.7k, Resistor_SMD:R_0402_1005Metric, F.Cu at (296.2, 247.8)
- added R18: 4.7k, Resistor_SMD:R_0402_1005Metric, F.Cu at (295.2, 247.8)
- added R19: 4.7k, Resistor_SMD:R_0402_1005Metric, F.Cu at (308.5, 241.2)
- added R20: 4.7k, Resistor_SMD:R_0402_1005Metric, F.Cu at (292.2, 248.0)
- added R202: 4.7k, KIT_Resistor_SMD:R_0603_1608Metric_DNP, F.Cu at (533.4, 170.6)
- added R21: 4.7k, Resistor_SMD:R_0402_1005Metric, F.Cu at (292.2, 247.0)
- added R22: 4.7k, Resistor_SMD:R_0402_1005Metric, F.Cu at (292.2, 238.5)
- added R23: 4.7k, Resistor_SMD:R_0402_1005Metric, F.Cu at (292.2, 237.5)
- added R24: 50, Resistor_SMD:R_0402_1005Metric, F.Cu at (293.7, 256.8)
- added R25: 50, Resistor_SMD:R_0402_1005Metric, F.Cu at (292.7, 256.8)
- added R26: 50, Resistor_SMD:R_0402_1005Metric, F.Cu at (296.7, 256.8)
- added R27: 50, Resistor_SMD:R_0402_1005Metric, F.Cu at (295.7, 256.8)
- added R28: 4.7k, Resistor_SMD:R_0402_1005Metric, F.Cu at (292.2, 273.0)
- added R29: 4.7k, Resistor_SMD:R_0402_1005Metric, F.Cu at (300.0, 272.8)
- added R30: 4.7k, Resistor_SMD:R_0402_1005Metric, F.Cu at (308.5, 266.2)
- added R31, R33: 4.7k, Resistor_SMD:R_0402_1005Metric, F.Cu at (292.2, 263.5)
- added R32: 4.7k, Resistor_SMD:R_0402_1005Metric, F.Cu at (295.2, 272.8)
- added R34: 4.7k, Resistor_SMD:R_0402_1005Metric, F.Cu at (296.2, 272.8)
- added R38: 10k, Resistor_SMD:R_2512_6332Metric, F.Cu at (480.5, 204.0)
- added R401: DNP, KIT_Resistor_SMD:R_0402_1005Metric_DNP, B.Cu at (520.5, 186.6)
- added R401: DNP, KIT_Resistor_SMD:R_0402_1005Metric_DNP, B.Cu at (525.4, 168.5)
- added R402: DNP, KIT_Resistor_SMD:R_0402_1005Metric_DNP, B.Cu at (520.5, 182.8)
- added R402: DNP, KIT_Resistor_SMD:R_0402_1005Metric_DNP, B.Cu at (525.4, 164.7)
- added R403: 0, KIT_Resistor_SMD:R_0402_1005Metric_DNP, B.Cu at (526.7, 168.5)
- added R403: 0, KIT_Resistor_SMD:R_0402_1005Metric_DNP, B.Cu at (521.7, 186.6)
- added R404: 0, Resistor_SMD:R_0402_1005Metric, B.Cu at (526.7, 164.7)
- added R404: 0, Resistor_SMD:R_0402_1005Metric, B.Cu at (521.7, 182.8)
- added R405: 11.3k, Resistor_SMD:R_0402_1005Metric, B.Cu at (521.6, 164.7)
- added R405: 11.3k, Resistor_SMD:R_0402_1005Metric, B.Cu at (516.7, 182.8)
- added R406: 11.5k, KIT_Resistor_SMD:R_0402_1005Metric_DNP, B.Cu at (520.3, 164.7)
- added R406: 11.5k, KIT_Resistor_SMD:R_0402_1005Metric_DNP, B.Cu at (515.4, 182.8)
- added R407: 10k, KIT_Resistor_SMD:R_0402_1005Metric_DNP, B.Cu at (517.2, 184.7)
- added R407: 10k, KIT_Resistor_SMD:R_0402_1005Metric_DNP, B.Cu at (522.2, 166.6)
- added R408: 0.1, Resistor_SMD:R_1210_3225Metric, B.Cu at (516.4, 167.6)
- added R409: 10, Resistor_SMD:R_0402_1005Metric, F.Cu at (512.5, 185.9)
- added R409: 10, Resistor_SMD:R_0402_1005Metric, F.Cu at (517.4, 167.8)
- added R41: 15, Resistor_SMD:R_2512_6332Metric, F.Cu at (337.7, 345.8)
- added R410: 10, Resistor_SMD:R_0402_1005Metric, F.Cu at (515.4, 167.8)
- added R42: 15, Resistor_SMD:R_2512_6332Metric, F.Cu at (332.0, 345.8)
- added R44: 0, Resistor_SMD:R_0402_1005Metric, F.Cu at (522.7, 189.9)
- added R46: 13.3k, Resistor_SMD:R_0402_1005Metric, F.Cu at (514.5, 182.7)
- added R47: 10k, Resistor_SMD:R_0402_1005Metric, F.Cu at (516.5, 178.4)
- added R51: 0, Resistor_SMD:R_0402_1005Metric, F.Cu at (483.2, 153.5)
- added R53: 30.1k, Resistor_SMD:R_0402_1005Metric, F.Cu at (483.2, 155.5)
- added R54: 10k, Resistor_SMD:R_0402_1005Metric, F.Cu at (483.2, 157.5)
- added TP1: TestPoint_Probe, TestPoint:TestPoint_Pad_D1.0mm, F.Cu at (524.2, 188.7)
- added TP2: TestPoint_Probe, TestPoint:TestPoint_Pad_D1.0mm, F.Cu at (478.8, 156.8)
- added TP202: TestPoint_Probe, TestPoint:TestPoint_Pad_D1.0mm, B.Cu at (530.4, 162.8)
- added TP401: TestPoint_Probe, TestPoint:TestPoint_Pad_D1.0mm, B.Cu at (528.4, 168.6)
- added TP401: TestPoint_Probe, TestPoint:TestPoint_Pad_D1.0mm, B.Cu at (523.5, 186.7)
- added TP502: TestPoint_Probe, TestPoint:TestPoint_Pad_D1.0mm, B.Cu at (514.7, 169.8)
- added U4: LTC4355, project:DFN-14_DE_LIT, F.Cu at (457.0, 302.5)
- added U401: LTM4624EY-PBF, Package_BGA:BGA-25_6.35x6.35mm_Layout5x5_P1.27mm, F.Cu at (524.2, 166.6)
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Connections:
- J14 pad 1: /SFP+/SC_SFP+_1.TX_DISABLE -> /SFP+/SC_SFP+.TX_DISABLE_1
- J15 pad 1: /SFP+/SC_SFP+_2.TX_DISABLE -> /SFP+/SC_SFP+.TX_DISABLE_2
- J6 pad 2: /SFP+/SC_SFP+_1.TX_FAULT -> /SFP+/SC_SFP+.TX_FAULT_1
- J6 pad 3: /SFP+/SC_SFP+_1.TX_DISABLE -> /SFP+/SC_SFP+.TX_DISABLE_1
- J6 pad 4: /SFP+/SC_SFP+_1.SDA -> /SFP+/SC_SFP+.SDA
- J6 pad 5: /SFP+/SC_SFP+_1.SCL -> /SFP+/SC_SFP+.SCL
- J6 pad 6: /SFP+/SC_SFP+_1.MOD_ABS -> /SFP+/SC_SFP+.MOD_ABS_1
- J6 pad 7: /SFP+/SC_SFP+_1.RS0 -> unconnected-(J6-RS0-Pad7)
- J6 pad 8: /SFP+/SC_SFP+_1.RX_LOS -> /SFP+/SC_SFP+.RX_LOS_1
- J6 pad 9: /SFP+/SC_SFP+_1.RS1 -> unconnected-(J6-RS1-Pad9)
- J7 pad 2: /SFP+/SC_SFP+_2.TX_FAULT -> /SFP+/SC_SFP+.TX_FAULT_2
- J7 pad 3: /SFP+/SC_SFP+_2.TX_DISABLE -> /SFP+/SC_SFP+.TX_DISABLE_2
- J7 pad 4: /SFP+/SC_SFP+_2.SDA -> /SFP+/SC_SFP+.SDA
- J7 pad 5: /SFP+/SC_SFP+_2.SCL -> /SFP+/SC_SFP+.SCL
- J7 pad 6: /SFP+/SC_SFP+_2.MOD_ABS -> /SFP+/SC_SFP+.MOD_ABS_2
- J7 pad 7: /SFP+/SC_SFP+_2.RS0 -> unconnected-(J7-RS0-Pad7)
- J7 pad 8: /SFP+/SC_SFP+_2.RX_LOS -> /SFP+/SC_SFP+.RX_LOS_2
- J7 pad 9: /SFP+/SC_SFP+_2.RS1 -> unconnected-(J7-RS1-Pad9)
- P10 pad 25: unconnected-(P10-SHELF_GND-Pad25) -> GNDPWR
- P10 pad 26: unconnected-(P10-LOGIC_GND-Pad26) -> GND
- P10 pad 28: unconnected-(P10-VRTN_A-Pad28) -> /ATCA_Z1/Z1_VRTN_A
- P10 pad 29: unconnected-(P10-VRTN_B-Pad29) -> /ATCA_Z1/Z1_VRTN_B
- P10 pad 30: unconnected-(P10-EARLY_A-Pad30) -> /ATCA_Z1/Z1_EARLY_A
- P10 pad 31: unconnected-(P10-EARLY_B-Pad31) -> /ATCA_Z1/Z1_EARLY_B
- P10 pad 33: unconnected-(P10-–48V_A-Pad33) -> /ATCA_Z1/Z1_-48V_A
- P10 pad 34: unconnected-(P10-–48V_B-Pad34) -> /ATCA_Z1/Z1_-48V_B
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Routing:
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- added copper zone on B.Cu, net (none)
- added copper zone on F.Cu, net (none)
- added copper zone on F.Cu, net +3V3
- added copper zone on F.Cu, net +5V
- added copper zone on In1.Cu, net /LHC_CLK/X1_guardring
- added copper zone on B.Cu, net GND
- added copper zone on F.Cu, net GND
Other:
- board size 99.9 x 193 mm -> 280 x 322.2 mm
- board text removed: "0"
- board text removed: "0 mm"
- board text removed: "0,01 mm"
- board text removed: "0,018 mm"
- board text removed: "0,02"
- board text removed: "0,035 mm"
- board text removed: "0,135 mm"
- board text removed: "0,2 mm"
- board text removed: "0,226 mm"
- board text removed: "1"
- board text removed: "3,3"
- board text removed: "4,6"
- board text removed: "B.Cu"
- board text removed: "B.Mask"
- board text removed: "B.Paste"
- board text removed: "B.Silkscreen"
- board text removed: "Bottom Silk Screen"
- board text removed: "Bottom Solder Mask"
- board text removed: "Bottom Solder Paste"
- board text removed: "Dicke (mm)"
- board text removed: "Dielektrikum"
- board text removed: "Epsilon R"
- board text removed: "F.Cu"
- board text removed: "F.Mask"
- board text removed: "F.Paste"
- board text removed: "F.Silkscreen"
- board text removed: "FR4"
- board text removed: "Farbe"
- board text removed: "Green"
- board text removed: "In10_GND.Cu"
- board text removed: "In1_GND.Cu"
- board text removed: "In2.Cu"
- board text removed: "In3_GND.Cu"
- board text removed: "In4.Cu"
- board text removed: "In5_PWR.Cu"
- board text removed: "In6_PWR.Cu"
- board text removed: "In7.Cu"
- board text removed: "In8_GND.Cu"
- board text removed: "In9.Cu"
- board text removed: "Lagenname"
- board text removed: "Material"
- board text removed: "Not specified"
- board text removed: "Top Silk Screen"
- board text removed: "Top Solder Mask"
- board text removed: "Top Solder Paste"
- board text removed: "Typ"
- board text removed: "Verlustwinkel"
- board text removed: "White"
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
Commit message: before sch review
Parts:
- removed C203, C205, C206, C208: 22uF, Capacitor_SMD:C_1210_3225Metric
- removed C401 (x2), C63: 10uF, Capacitor_SMD:C_0603_1608Metric
- removed C402 (x2), C403 (x2), C64, C65: 10uF, Capacitor_SMD:C_0805_2012Metric
- removed C404 (x2): 1uF, Capacitor_SMD:C_0402_1005Metric
- removed C405 (x2): 0.1uF, Capacitor_SMD:C_0402_1005Metric
- removed C406 (x2), C407: 47uF, Capacitor_SMD:C_0805_2012Metric
- removed C408: C, Capacitor_SMD:C_0402_1005Metric
- removed C56: 4700pF, project:VISAY_CAP_MY5UCR
- removed D1, D2, D3: BAS21, Package_TO_SOT_SMD:SOT-23
- removed D4: SMBJ5347B-TP, project:SMBJ5347B-TP_DO-214AA
- removed J15: Conn_01x02_Pin, Connector_PinHeader_2.54mm:PinHeader_1x02_P2.54mm_Vertical
- removed L1, L2, L401 (x2): BLM18SG121TZ1D, Inductor_SMD:L_0603_1608Metric
- removed NT401 (x2): Net-Tie_2, KIT_NetTie:NetTie-2_SMD_Pad0.3mm
- removed Q1, Q2, Q3, Q4: IRF3710Z, project:D2PAK_TO-263AB_INF
- removed R202: 4.7k, KIT_Resistor_SMD:R_0603_1608Metric_DNP
- removed R38: 10k, Resistor_SMD:R_2512_6332Metric
- removed R401 (x2), R402 (x2): DNP, KIT_Resistor_SMD:R_0402_1005Metric_DNP
- removed R403 (x2): 0, KIT_Resistor_SMD:R_0402_1005Metric_DNP
- removed R404 (x2), R44, R51: 0, Resistor_SMD:R_0402_1005Metric
- removed R405 (x2): 11.3k, Resistor_SMD:R_0402_1005Metric
- removed R406 (x2): 11.5k, KIT_Resistor_SMD:R_0402_1005Metric_DNP
- removed R407 (x2): 10k, KIT_Resistor_SMD:R_0402_1005Metric_DNP
- removed R408: 0.1, Resistor_SMD:R_1210_3225Metric
- removed R409 (x2), R410: 10, Resistor_SMD:R_0402_1005Metric
- removed R46: 13.3k, Resistor_SMD:R_0402_1005Metric
- removed R47, R54: 10k, Resistor_SMD:R_0402_1005Metric
- removed R53: 30.1k, Resistor_SMD:R_0402_1005Metric
- removed TP1, TP2, TP202, TP401 (x2), TP502: TestPoint_Probe, TestPoint:TestPoint_Pad_D1.0mm
- removed U401, U8, U9: LTM4624EY-PBF, Package_BGA:BGA-25_6.35x6.35mm_Layout5x5_P1.27mm
- removed U6: PDQE20-Q48-S5-D, project:CUI_PDQE20-Q48-S5-D
- removed U7: LTC4354, project:DFN-8_DDB_LIT
- added A1: FrontPanel, KIT_Mechanical:FrontPanel, F.Cu at (95.0, 193.5)
- added C100: 100nF, Capacitor_SMD:C_0402_1005Metric, F.Cu at (435.4, 314.6)
- added C51: 22uF, Capacitor_SMD:C_0805_2012Metric, F.Cu at (430.5, 327.6)
- added C61: 20nF, Capacitor_SMD:C_0805_2012Metric, F.Cu at (423.7, 307.3)
- added C77: 20nF, Capacitor_SMD:C_0805_2012Metric, F.Cu at (423.7, 310.3)
- added C78: 20nF, Capacitor_SMD:C_0805_2012Metric, F.Cu at (423.7, 313.3)
- added C79: 100uF, Capacitor_THT:CP_Radial_D16.0mm_P7.50mm, F.Cu at (409.0, 314.6)
- added C80: 100uF, Capacitor_THT:CP_Radial_D16.0mm_P7.50mm, F.Cu at (409.0, 332.1)
- added C81: 100uF, Capacitor_THT:CP_Radial_D16.0mm_P7.50mm, F.Cu at (409.0, 349.7)
- added C82: 22uF, Capacitor_SMD:C_0805_2012Metric, F.Cu at (423.7, 316.3)
- added C83: 100nF, Capacitor_SMD:C_0402_1005Metric, F.Cu at (429.7, 306.8)
- added C84: 22uF, Capacitor_SMD:C_0805_2012Metric, F.Cu at (423.7, 319.3)
- added C85: 100nF, Capacitor_SMD:C_0402_1005Metric, F.Cu at (429.7, 308.7)
- added C86: 100nF, Capacitor_SMD:C_0402_1005Metric, F.Cu at (429.7, 310.7)
- added C87: 100nF, Capacitor_SMD:C_0402_1005Metric, F.Cu at (429.7, 312.7)
- added C88: 100nF, Capacitor_SMD:C_0402_1005Metric, F.Cu at (429.7, 314.6)
- added C89: 100nF, Capacitor_SMD:C_0402_1005Metric, F.Cu at (429.7, 316.6)
- added C90: 100nF, Capacitor_SMD:C_0402_1005Metric, F.Cu at (432.6, 306.8)
- added C91: 100nF, Capacitor_SMD:C_0402_1005Metric, F.Cu at (432.6, 308.7)
- added C92: 100nF, Capacitor_SMD:C_0402_1005Metric, F.Cu at (432.6, 310.7)
- added C93: 100nF, Capacitor_SMD:C_0402_1005Metric, F.Cu at (432.6, 312.7)
- added C94: 100nF, Capacitor_SMD:C_0402_1005Metric, F.Cu at (432.6, 314.6)
- added C95: 100nF, Capacitor_SMD:C_0402_1005Metric, F.Cu at (432.6, 316.6)
- added C96: 100nF, Capacitor_SMD:C_0402_1005Metric, F.Cu at (435.4, 306.8)
- added C97: 100nF, Capacitor_SMD:C_0402_1005Metric, F.Cu at (435.4, 308.7)
- added C98: 100nF, Capacitor_SMD:C_0402_1005Metric, F.Cu at (435.4, 310.7)
- added C99: 100nF, Capacitor_SMD:C_0402_1005Metric, F.Cu at (435.4, 312.7)
- added F1: 1A, project:SM2410, F.Cu at (393.9, 366.8)
- added F2: 15A, project:SM2410, F.Cu at (393.9, 372.0)
- added F3: 15A, project:SM2410, F.Cu at (393.9, 377.3)
- added F4: 1A, project:SM2410, F.Cu at (393.9, 382.5)
- added F5: 15A, project:SM2410, F.Cu at (393.9, 387.7)
- added F6: 15A, project:SM2410, F.Cu at (393.9, 392.9)
- added H1: 81-088-1, KIT_Mechanical:81-301-00, F.Cu at (100.0, 350.0)
- added H2: Handle, project:81-300-00, F.Cu at (100.0, 38.9)
- added J17: Conn_01x03_Pin, Connector_PinHeader_2.54mm:PinHeader_1x03_P2.54mm_Vertical, F.Cu at (108.2, 77.8)
- added K1: Key_K1_K2_TE_1-1469373-1, project:Key_K1_K2_TE_1-1469373-1, F.Cu at (354.1, 63.5)
- added NT1: Net-Tie_2, NetTie:NetTie-2_SMD_Pad0.5mm, F.Cu at (123.5, 123.4)
- added Q5: DMG2305UX, Package_TO_SOT_SMD:TSOT-23, F.Cu at (431.0, 321.8)
- added R35: 10k, Resistor_SMD:R_0805_2012Metric, F.Cu at (400.4, 365.7)
- added R37: 10k, Resistor_SMD:R_0603_1608Metric, F.Cu at (344.6, 72.8)
- added R7: 2k2, Resistor_SMD:R_0805_2012Metric_Pad1.20x1.40mm_HandSolder, F.Cu at (423.9, 322.3)
- added R8: 4k7, Resistor_SMD:R_0402_1005Metric, F.Cu at (423.0, 324.8)
- C49: value 4700pF -> 22uF; footprint project:VISAY_CAP_MY5UCR -> Capacitor_SMD:C_0805_2012Metric
- C50: value 47uF -> 1nF; footprint project:CHEMI-KE0 -> Capacitor_SMD:C_0402_1005Metric
- C52, C53, C54: value 4700pF -> 100nF; footprint project:VISAY_CAP_MY5UCR -> Capacitor_SMD:C_0402_1005Metric
- C55: value 47uF -> 100nF; footprint project:CHEMI-KE0 -> Capacitor_SMD:C_0402_1005Metric
- C62: value 4700pF -> 20nF; footprint project:VISAY_CAP_MY5UCR -> Capacitor_SMD:C_0805_2012Metric
- C66, C73: value 1uF -> 100nF
- C67, C74: value 0.1uF -> 100nF
- C68, C69, C75, C76: value 47uF -> 100nF; footprint Capacitor_SMD:C_0805_2012Metric -> Capacitor_SMD:C_0402_1005Metric
- C70: value 10uF -> 100nF; footprint Capacitor_SMD:C_0603_1608Metric -> Capacitor_SMD:C_0402_1005Metric
- C71, C72: value 10uF -> 100nF; footprint Capacitor_SMD:C_0805_2012Metric -> Capacitor_SMD:C_0402_1005Metric
- J14: value Conn_01x02_Pin -> Conn_01x03_Male; footprint Connector_PinHeader_2.54mm:PinHeader_1x02_P2.54mm_Vertical -> KIT_Connector:Molex_53046-0310
- J3: footprint project:ESD_strip_bottom -> project:ESD_Strip
- U4: value LTC4355 -> PIM400KZ; footprint project:DFN-14_DE_LIT -> project:PIM400KZ
- U5: value QPI-21LZ-01 -> ADM7172; footprint project:VICOR_QPI-21 LGA_OPEN -> Package_CSP:LFCSP-8-1EP_3x3mm_P0.5mm_EP1.45x1.74mm
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Connections:
- net /SFP+/SC_SFP+.MOD_ABS_1 renamed /SFP+/SC_SFP+_1.MOD_ABS_1
- net /SFP+/SC_SFP+.MOD_ABS_2 renamed /SFP+/SC_SFP+_2.MOD_ABS_2
- net /SFP+/SC_SFP+.RX_LOS_1 renamed /SFP+/SC_SFP+_1.RX_LOS_1
- net /SFP+/SC_SFP+.RX_LOS_2 renamed /SFP+/SC_SFP+_1.RX_LOS_2
- net /SFP+/SC_SFP+.TX_FAULT_1 renamed /SFP+/SC_SFP+_1.TX_FAULT_1
- net /SFP+/SC_SFP+.TX_FAULT_2 renamed /SFP+/SC_SFP+_2.TX_FAULT_2
- C49 pad 1: Net-(D4-A) -> +3V3
- C49 pad 2: GNDPWR -> GND
- C50 pad 1: Net-(U5-XY+) -> Net-(U5-SS)
- C50 pad 2: Net-(U5-XY-) -> GND
- C52 pad 1: Net-(U6-VIN) -> Net-(J1A-TRCT1_1)
- C52 pad 2: GNDPWR -> GND
- C53 pad 1: GND -> Net-(J1A-TRCT2_1)
- C53 pad 2: GNDPWR -> GND
- C54 pad 1: +5V -> Net-(J1A-TRCT3_1)
- C54 pad 2: GNDPWR -> GND
- C55 pad 1: Net-(U6-VIN) -> Net-(J1A-TRCT4_1)
- C55 pad 2: Net-(D4-A) -> GND
- C57 pad 1: /ATCA_Z1/BUS_A_P -> /ATCA_Z1/PIM400_VRET_A
- C57 pad 2: /ATCA_Z1/BUS_A_N -> /ATCA_Z1/PIM400_-48V_A
- C58 pad 1: /ATCA_Z1/BUS_B_P -> /ATCA_Z1/PIM400_VRET_B
- C58 pad 2: /ATCA_Z1/BUS_B_N -> /ATCA_Z1/PIM400_-48V_B
- C59 pad 1: /ATCA_Z1/BUS_A_P -> /ATCA_Z1/PIM400_VRET_A
- C59 pad 2: /ATCA_Z1/BUS_A_N -> /ATCA_Z1/PIM400_-48V_A
- C60 pad 1: /ATCA_Z1/BUS_B_P -> /ATCA_Z1/PIM400_VRET_B
- C60 pad 2: /ATCA_Z1/BUS_B_N -> /ATCA_Z1/PIM400_-48V_B
- C62 pad 1: +5V -> /ATCA_Z1/PIM400_Shield_Plane
- C66 pad 1: /Power 3V3/INTVCC -> Net-(J1B-TRCT1_2)
- C67 pad 1: /Power 3V3/SS -> Net-(J1B-TRCT2_2)
- C67 pad 2: /Power 3V3/SGND -> GND
- C68 pad 1: +3V3 -> Net-(J1B-TRCT3_2)
- C69 pad 1: +3V3 -> Net-(J1B-TRCT4_2)
- C70 pad 1: +5V -> Net-(J1D-TRCT1_4)
- C71 pad 1: /Power 1V8/VIN -> Net-(J1D-TRCT2_4)
- C72 pad 1: /Power 1V8/VIN -> Net-(J1D-TRCT3_4)
- C73 pad 1: /Power 1V8/INTVCC -> Net-(J1D-TRCT4_4)
- C74 pad 1: /Power 1V8/SS -> Net-(J1C-TRCT1_3)
- C74 pad 2: /Power 1V8/SGND -> GND
- C75 pad 1: +1V8 -> Net-(J1C-TRCT2_3)
- C76 pad 1: +1V8 -> Net-(J1C-TRCT3_3)
- J1 pad 10_1: unconnected-(J1A-TRD1-_1-Pad10_1) -> /Z2_BI1.A_N
- J1 pad 10_2: unconnected-(J1B-TRD1-_2-Pad10_2) -> /Z2_BI2.A_N
- J1 pad 10_3: unconnected-(J1C-TRD1-_3-Pad10_3) -> /Z2_BI4.A_N
- J1 pad 10_4: unconnected-(J1D-TRD1-_4-Pad10_4) -> /Z2_BI3.A_N
- J1 pad 11_1: unconnected-(J1A-TRD1+_1-Pad11_1) -> /Z2_BI1.A_P
- J1 pad 11_2: unconnected-(J1B-TRD1+_2-Pad11_2) -> /Z2_BI2.A_P
- J1 pad 11_3: unconnected-(J1C-TRD1+_3-Pad11_3) -> /Z2_BI4.A_P
- J1 pad 11_4: unconnected-(J1D-TRD1+_4-Pad11_4) -> /Z2_BI3.A_P
- J1 pad 12_1: unconnected-(J1A-TRCT1_1-Pad12_1) -> Net-(J1A-TRCT1_1)
- J1 pad 12_2: unconnected-(J1B-TRCT1_2-Pad12_2) -> Net-(J1B-TRCT1_2)
- J1 pad 12_3: unconnected-(J1C-TRCT1_3-Pad12_3) -> Net-(J1C-TRCT1_3)
- J1 pad 12_4: unconnected-(J1D-TRCT1_4-Pad12_4) -> Net-(J1D-TRCT1_4)
- J1 pad 1_1: unconnected-(J1A-TRCT3_1-Pad1_1) -> Net-(J1A-TRCT3_1)
- J1 pad 1_2: unconnected-(J1B-TRCT3_2-Pad1_2) -> Net-(J1B-TRCT3_2)
- J1 pad 1_3: unconnected-(J1C-TRCT3_3-Pad1_3) -> Net-(J1C-TRCT3_3)
- J1 pad 1_4: unconnected-(J1D-TRCT3_4-Pad1_4) -> Net-(J1D-TRCT3_4)
- J1 pad 2_1: unconnected-(J1A-TRD3-_1-Pad2_1) -> /Z2_BI1.C_N
- J1 pad 2_2: unconnected-(J1B-TRD3-_2-Pad2_2) -> /Z2_BI2.C_N
- J1 pad 2_3: unconnected-(J1C-TRD3-_3-Pad2_3) -> /Z2_BI4.C_N
- J1 pad 2_4: unconnected-(J1D-TRD3-_4-Pad2_4) -> /Z2_BI3.C_N
- J1 pad 3_1: unconnected-(J1A-TRD3+_1-Pad3_1) -> /Z2_BI1.C_P
- J1 pad 3_2: unconnected-(J1B-TRD3+_2-Pad3_2) -> /Z2_BI2.C_P
- J1 pad 3_3: unconnected-(J1C-TRD3+_3-Pad3_3) -> /Z2_BI4.C_P
- J1 pad 3_4: unconnected-(J1D-TRD3+_4-Pad3_4) -> /Z2_BI3.C_P
- J1 pad 4_1: unconnected-(J1A-TRD2+_1-Pad4_1) -> /Z2_BI1.B_P
- J1 pad 4_2: unconnected-(J1B-TRD2+_2-Pad4_2) -> /Z2_BI2.B_P
- J1 pad 4_3: unconnected-(J1C-TRD2+_3-Pad4_3) -> /Z2_BI4.B_P
- J1 pad 4_4: unconnected-(J1D-TRD2+_4-Pad4_4) -> /Z2_BI3.B_P
- J1 pad 5_1: unconnected-(J1A-TRD2-_1-Pad5_1) -> /Z2_BI1.B_N
- J1 pad 5_2: unconnected-(J1B-TRD2-_2-Pad5_2) -> /Z2_BI2.B_N
- J1 pad 5_3: unconnected-(J1C-TRD2-_3-Pad5_3) -> /Z2_BI4.B_N
- J1 pad 5_4: unconnected-(J1D-TRD2-_4-Pad5_4) -> /Z2_BI3.B_N
- J1 pad 6_1: unconnected-(J1A-TRCT2_1-Pad6_1) -> Net-(J1A-TRCT2_1)
- J1 pad 6_2: unconnected-(J1B-TRCT2_2-Pad6_2) -> Net-(J1B-TRCT2_2)
- J1 pad 6_3: unconnected-(J1C-TRCT2_3-Pad6_3) -> Net-(J1C-TRCT2_3)
- J1 pad 6_4: unconnected-(J1D-TRCT2_4-Pad6_4) -> Net-(J1D-TRCT2_4)
- J1 pad 7_1: unconnected-(J1A-TRCT4_1-Pad7_1) -> Net-(J1A-TRCT4_1)
- J1 pad 7_2: unconnected-(J1B-TRCT4_2-Pad7_2) -> Net-(J1B-TRCT4_2)
- J1 pad 7_3: unconnected-(J1C-TRCT4_3-Pad7_3) -> Net-(J1C-TRCT4_3)
- J1 pad 7_4: unconnected-(J1D-TRCT4_4-Pad7_4) -> Net-(J1D-TRCT4_4)
- J1 pad 8_1: unconnected-(J1A-TRD4+_1-Pad8_1) -> /Z2_BI1.D_P
- J1 pad 8_2: unconnected-(J1B-TRD4+_2-Pad8_2) -> /Z2_BI2.D_P
- J1 pad 8_3: unconnected-(J1C-TRD4+_3-Pad8_3) -> /Z2_BI4.D_P
- J1 pad 8_4: unconnected-(J1D-TRD4+_4-Pad8_4) -> /Z2_BI3.D_P
- J1 pad 9_1: unconnected-(J1A-TRD4-_1-Pad9_1) -> /Z2_BI1.D_N
- J1 pad 9_2: unconnected-(J1B-TRD4-_2-Pad9_2) -> /Z2_BI2.D_N
- J1 pad 9_3: unconnected-(J1C-TRD4-_3-Pad9_3) -> /Z2_BI4.D_N
- J1 pad 9_4: unconnected-(J1D-TRD4-_4-Pad9_4) -> /Z2_BI3.D_N
- J1 pad S1: Net-(J1A-SHIELD-PadS1) -> GNDPWR
- J1 pad S2: Net-(J1A-SHIELD-PadS1) -> GNDPWR
- J14 pad 1: /SFP+/SC_SFP+.TX_DISABLE_1 -> FP_HANDLE
- J2 pad 10_1: unconnected-(J2A-TRD1-_1-Pad10_1) -> /Z2_BI5.A_N
- J2 pad 10_2: unconnected-(J2B-TRD1-_2-Pad10_2) -> /Z2_BI6.A_N
- J2 pad 10_3: unconnected-(J2C-TRD1-_3-Pad10_3) -> /Z2_BI8.A_N
- J2 pad 10_4: unconnected-(J2D-TRD1-_4-Pad10_4) -> /Z2_BI7.A_N
- J2 pad 11_1: unconnected-(J2A-TRD1+_1-Pad11_1) -> /Z2_BI5.A_P
- J2 pad 11_2: unconnected-(J2B-TRD1+_2-Pad11_2) -> /Z2_BI6.A_P
- J2 pad 11_3: unconnected-(J2C-TRD1+_3-Pad11_3) -> /Z2_BI8.A_P
- J2 pad 11_4: unconnected-(J2D-TRD1+_4-Pad11_4) -> /Z2_BI7.A_P
- J2 pad 12_1: unconnected-(J2A-TRCT1_1-Pad12_1) -> Net-(J2A-TRCT1_1)
- J2 pad 12_2: unconnected-(J2B-TRCT1_2-Pad12_2) -> Net-(J2B-TRCT1_2)
- J2 pad 12_3: unconnected-(J2C-TRCT1_3-Pad12_3) -> Net-(J2C-TRCT1_3)
- J2 pad 12_4: unconnected-(J2D-TRCT1_4-Pad12_4) -> Net-(J2D-TRCT1_4)
- J2 pad 1_1: unconnected-(J2A-TRCT3_1-Pad1_1) -> Net-(J2A-TRCT3_1)
- J2 pad 1_2: unconnected-(J2B-TRCT3_2-Pad1_2) -> Net-(J2B-TRCT3_2)
- J2 pad 1_3: unconnected-(J2C-TRCT3_3-Pad1_3) -> Net-(J2C-TRCT3_3)
- J2 pad 1_4: unconnected-(J2D-TRCT3_4-Pad1_4) -> Net-(J2D-TRCT3_4)
- J2 pad 2_1: unconnected-(J2A-TRD3-_1-Pad2_1) -> /Z2_BI5.C_N
- J2 pad 2_2: unconnected-(J2B-TRD3-_2-Pad2_2) -> /Z2_BI6.C_N
- J2 pad 2_3: unconnected-(J2C-TRD3-_3-Pad2_3) -> /Z2_BI8.C_N
- J2 pad 2_4: unconnected-(J2D-TRD3-_4-Pad2_4) -> /Z2_BI7.C_N
- J2 pad 3_1: unconnected-(J2A-TRD3+_1-Pad3_1) -> /Z2_BI5.C_P
- J2 pad 3_2: unconnected-(J2B-TRD3+_2-Pad3_2) -> /Z2_BI6.C_P
- J2 pad 3_3: unconnected-(J2C-TRD3+_3-Pad3_3) -> /Z2_BI8.C_P
- J2 pad 3_4: unconnected-(J2D-TRD3+_4-Pad3_4) -> /Z2_BI7.C_P
- J2 pad 4_1: unconnected-(J2A-TRD2+_1-Pad4_1) -> /Z2_BI5.B_P
- J2 pad 4_2: unconnected-(J2B-TRD2+_2-Pad4_2) -> /Z2_BI6.B_P
- J2 pad 4_3: unconnected-(J2C-TRD2+_3-Pad4_3) -> /Z2_BI8.B_P
- J2 pad 4_4: unconnected-(J2D-TRD2+_4-Pad4_4) -> /Z2_BI7.B_P
- J2 pad 5_1: unconnected-(J2A-TRD2-_1-Pad5_1) -> /Z2_BI5.B_N
- J2 pad 5_2: unconnected-(J2B-TRD2-_2-Pad5_2) -> /Z2_BI6.B_N
- J2 pad 5_3: unconnected-(J2C-TRD2-_3-Pad5_3) -> /Z2_BI8.B_N
- J2 pad 5_4: unconnected-(J2D-TRD2-_4-Pad5_4) -> /Z2_BI7.B_N
- J2 pad 6_1: unconnected-(J2A-TRCT2_1-Pad6_1) -> Net-(J2A-TRCT2_1)
- J2 pad 6_2: unconnected-(J2B-TRCT2_2-Pad6_2) -> Net-(J2B-TRCT2_2)
- J2 pad 6_3: unconnected-(J2C-TRCT2_3-Pad6_3) -> Net-(J2C-TRCT2_3)
- J2 pad 6_4: unconnected-(J2D-TRCT2_4-Pad6_4) -> Net-(J2D-TRCT2_4)
- J2 pad 7_1: unconnected-(J2A-TRCT4_1-Pad7_1) -> Net-(J2A-TRCT4_1)
- J2 pad 7_2: unconnected-(J2B-TRCT4_2-Pad7_2) -> Net-(J2B-TRCT4_2)
- J2 pad 7_3: unconnected-(J2C-TRCT4_3-Pad7_3) -> Net-(J2C-TRCT4_3)
- J2 pad 7_4: unconnected-(J2D-TRCT4_4-Pad7_4) -> Net-(J2D-TRCT4_4)
- J2 pad 8_1: unconnected-(J2A-TRD4+_1-Pad8_1) -> /Z2_BI5.D_P
- J2 pad 8_2: unconnected-(J2B-TRD4+_2-Pad8_2) -> /Z2_BI6.D_P
- J2 pad 8_3: unconnected-(J2C-TRD4+_3-Pad8_3) -> /Z2_BI8.D_P
- J2 pad 8_4: unconnected-(J2D-TRD4+_4-Pad8_4) -> /Z2_BI7.D_P
- J2 pad 9_1: unconnected-(J2A-TRD4-_1-Pad9_1) -> /Z2_BI5.D_N
- J2 pad 9_2: unconnected-(J2B-TRD4-_2-Pad9_2) -> /Z2_BI6.D_N
- J2 pad 9_3: unconnected-(J2C-TRD4-_3-Pad9_3) -> /Z2_BI8.D_N
- J2 pad 9_4: unconnected-(J2D-TRD4-_4-Pad9_4) -> /Z2_BI7.D_N
- J2 pad S1: Net-(J2A-SHIELD-PadS1) -> GNDPWR
- J2 pad S2: Net-(J2A-SHIELD-PadS1) -> GNDPWR
- J6 pad 3: /SFP+/SC_SFP+.TX_DISABLE_1 -> /SFP+/SC_SFP+_1.TX_DISABLE_1
- J6 pad 4: /SFP+/SC_SFP+.SDA -> /ATCA_Z1/SC_PIM.SDA
- J6 pad 5: /SFP+/SC_SFP+.SCL -> /ATCA_Z1/SC_PIM.SCL
- J7 pad 3: /SFP+/SC_SFP+.TX_DISABLE_2 -> /SFP+/SC_SFP+_2.TX_DISABLE_2
- J7 pad 4: /SFP+/SC_SFP+.SDA -> /LHC_CLK/SC_PLL.SDA
- J7 pad 5: /SFP+/SC_SFP+.SCL -> /LHC_CLK/SC_PLL.SCL
- P10 pad 27: unconnected-(P10-ENABLE_B-Pad27) -> /ATCA_Z1/Z1_EN_B
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Routing:
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- added copper zone on In1.Cu, net /LHC_CLK_HQ/X1_guardring
- removed copper zone on B.Cu, net (none)
- removed copper zone on F.Cu, net (none)
- removed copper zone on F.Cu, net +3V3
- removed copper zone on F.Cu, net +5V
- removed copper zone on B.Cu, net GND
- removed copper zone on F.Cu, net GND

Commit message: started changes from review
Parts:
- C57, C58, C59, C60, R41, R42, R7: moved to B.Cu
- C79, C80, C81: footprint Capacitor_THT:CP_Radial_D16.0mm_P7.50mm -> Capacitor_SMD:CP_Elec_18x22
- moved Q5 411.6 mm to (102.3, 74.0)
- moved C73 377.5 mm to (126.2, 254.0)
- moved C74 377.3 mm to (126.7, 257.0)
- moved C76 371.1 mm to (126.5, 268.0)
- moved C68 370.5 mm to (126.5, 280.5)
- moved C70 370.3 mm to (126.8, 241.0)
- moved C69 369.9 mm to (126.5, 281.5)
- moved C75 368.7 mm to (126.7, 258.0)
- moved C72 368.3 mm to (126.5, 252.8)
- moved C71 366.0 mm to (126.7, 242.2)
- moved C52 337.0 mm to (126.8, 285.0)
- moved C53 333.6 mm to (126.7, 286.0)
- moved C54 333.2 mm to (126.8, 295.2)
- moved C93 332.4 mm to (127.8, 180.0)
- moved C94 332.4 mm to (127.8, 182.0)
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Connections:
- C61 pad 2: GND -> GNDPWR
- C62 pad 2: GND -> GNDPWR
- C77 pad 2: GND -> GNDPWR
- C78 pad 2: GND -> GNDPWR
- J1 pad 10_1: /Z2_BI1.A_N -> /Z2_BI8.A_N
- J1 pad 10_2: /Z2_BI2.A_N -> /Z2_BI7.A_N
- J1 pad 10_3: /Z2_BI4.A_N -> /Z2_BI6.A_N
- J1 pad 10_4: /Z2_BI3.A_N -> /Z2_BI5.A_N
- J1 pad 11_1: /Z2_BI1.A_P -> /Z2_BI8.A_P
- J1 pad 11_2: /Z2_BI2.A_P -> /Z2_BI7.A_P
- J1 pad 11_3: /Z2_BI4.A_P -> /Z2_BI6.A_P
- J1 pad 11_4: /Z2_BI3.A_P -> /Z2_BI5.A_P
- J1 pad 2_1: /Z2_BI1.C_N -> /Z2_BI8.C_N
- J1 pad 2_2: /Z2_BI2.C_N -> /Z2_BI7.C_N
- J1 pad 2_3: /Z2_BI4.C_N -> /Z2_BI6.C_N
- J1 pad 2_4: /Z2_BI3.C_N -> /Z2_BI5.C_N
- J1 pad 3_1: /Z2_BI1.C_P -> /Z2_BI8.C_P
- J1 pad 3_2: /Z2_BI2.C_P -> /Z2_BI7.C_P
- J1 pad 3_3: /Z2_BI4.C_P -> /Z2_BI6.C_P
- J1 pad 3_4: /Z2_BI3.C_P -> /Z2_BI5.C_P
- J1 pad 4_1: /Z2_BI1.B_P -> /Z2_BI8.B_P
- J1 pad 4_2: /Z2_BI2.B_P -> /Z2_BI7.B_P
- J1 pad 4_3: /Z2_BI4.B_P -> /Z2_BI6.B_P
- J1 pad 4_4: /Z2_BI3.B_P -> /Z2_BI5.B_P
- J1 pad 5_1: /Z2_BI1.B_N -> /Z2_BI8.B_N
- J1 pad 5_2: /Z2_BI2.B_N -> /Z2_BI7.B_N
- J1 pad 5_3: /Z2_BI4.B_N -> /Z2_BI6.B_N
- J1 pad 5_4: /Z2_BI3.B_N -> /Z2_BI5.B_N
- J1 pad 8_1: /Z2_BI1.D_P -> /Z2_BI8.D_P
- J1 pad 8_2: /Z2_BI2.D_P -> /Z2_BI7.D_P
- J1 pad 8_3: /Z2_BI4.D_P -> /Z2_BI6.D_P
- J1 pad 8_4: /Z2_BI3.D_P -> /Z2_BI5.D_P
- J1 pad 9_1: /Z2_BI1.D_N -> /Z2_BI8.D_N
- J1 pad 9_2: /Z2_BI2.D_N -> /Z2_BI7.D_N
- J1 pad 9_3: /Z2_BI4.D_N -> /Z2_BI6.D_N
- J1 pad 9_4: /Z2_BI3.D_N -> /Z2_BI5.D_N
- J2 pad 10_1: /Z2_BI5.A_N -> /Z2_BI4.A_N
- J2 pad 10_2: /Z2_BI6.A_N -> /Z2_BI3.A_N
- J2 pad 10_3: /Z2_BI8.A_N -> /Z2_BI2.A_N
- J2 pad 10_4: /Z2_BI7.A_N -> /Z2_BI1.A_N
- J2 pad 11_1: /Z2_BI5.A_P -> /Z2_BI4.A_P
- J2 pad 11_2: /Z2_BI6.A_P -> /Z2_BI3.A_P
- J2 pad 11_3: /Z2_BI8.A_P -> /Z2_BI2.A_P
- J2 pad 11_4: /Z2_BI7.A_P -> /Z2_BI1.A_P
- J2 pad 2_1: /Z2_BI5.C_N -> /Z2_BI4.C_N
- J2 pad 2_2: /Z2_BI6.C_N -> /Z2_BI3.C_N
- J2 pad 2_3: /Z2_BI8.C_N -> /Z2_BI2.C_N
- J2 pad 2_4: /Z2_BI7.C_N -> /Z2_BI1.C_N
- J2 pad 3_1: /Z2_BI5.C_P -> /Z2_BI4.C_P
- J2 pad 3_2: /Z2_BI6.C_P -> /Z2_BI3.C_P
- J2 pad 3_3: /Z2_BI8.C_P -> /Z2_BI2.C_P
- J2 pad 3_4: /Z2_BI7.C_P -> /Z2_BI1.C_P
- J2 pad 4_1: /Z2_BI5.B_P -> /Z2_BI4.B_P
- J2 pad 4_2: /Z2_BI6.B_P -> /Z2_BI3.B_P
- J2 pad 4_3: /Z2_BI8.B_P -> /Z2_BI2.B_P
- J2 pad 4_4: /Z2_BI7.B_P -> /Z2_BI1.B_P
- J2 pad 5_1: /Z2_BI5.B_N -> /Z2_BI4.B_N
- J2 pad 5_2: /Z2_BI6.B_N -> /Z2_BI3.B_N
- J2 pad 5_3: /Z2_BI8.B_N -> /Z2_BI2.B_N
- J2 pad 5_4: /Z2_BI7.B_N -> /Z2_BI1.B_N
- J2 pad 8_1: /Z2_BI5.D_P -> /Z2_BI4.D_P
- J2 pad 8_2: /Z2_BI6.D_P -> /Z2_BI3.D_P
- J2 pad 8_3: /Z2_BI8.D_P -> /Z2_BI2.D_P
- J2 pad 8_4: /Z2_BI7.D_P -> /Z2_BI1.D_P
- J2 pad 9_1: /Z2_BI5.D_N -> /Z2_BI4.D_N
- J2 pad 9_2: /Z2_BI6.D_N -> /Z2_BI3.D_N
- J2 pad 9_3: /Z2_BI8.D_N -> /Z2_BI2.D_N
- J2 pad 9_4: /Z2_BI7.D_N -> /Z2_BI1.D_N
Routing:
- net /Z2_BI1.A_P: track 0.00 -> 186.9 mm
- net /Z2_BI1.A_N: track 0.00 -> 185.9 mm
- net /Z2_FI1.LHC_CLK_HQ_P: track 0.00 -> 80.9 mm
- net /Z2_FI1.LHC_CLK_HQ_N: track 0.00 -> 79.7 mm
- net /Z2_FI2.LHC_CLK_HQ_P: track 0.00 -> 72.6 mm
- net /Z2_FI2.LHC_CLK_HQ_N: track 0.00 -> 71.9 mm
- net /Z2_FI3.LHC_CLK_HQ_P: track 0.00 -> 67.7 mm
- net /Z2_FI3.LHC_CLK_HQ_N: track 0.00 -> 67.3 mm
- net /Z2_FI4.LHC_CLK_HQ_P: track 0.00 -> 66.2 mm
- net /Z2_FI4.LHC_CLK_HQ_N: track 0.00 -> 65.9 mm
- net /Z2_FI6.LHC_CLK_HQ_P: track 0.00 -> 16.1 mm
- net /Z2_FI7.LHC_CLK_HQ_P: track 0.00 -> 16.1 mm
- net /J22/10GbE_RX_P: track 0.00 -> 16.0 mm
- net /LHC_CLK/FB_CLK_N: track 0.00 -> 15.9 mm
- net /LHC_CLK_HQ/FB_CLK_N: track 0.00 -> 15.9 mm
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- added copper zone on F.Cu, net /ATCA_Z1/PIM400_Shield_Plane
Other:
- copper layers 12 -> 8

Commit message: starting doing stackup calculations
Parts:
- removed J17: Conn_01x03_Pin, Connector_PinHeader_2.54mm:PinHeader_1x03_P2.54mm_Vertical
- added C101: 1uF, Capacitor_SMD:C_0402_1005Metric, F.Cu at (313.6, 104.3)
- added C102: 10uF, Capacitor_SMD:C_0603_1608Metric, F.Cu at (308.2, 110.1)
- added C103: 1uF, Capacitor_SMD:C_0402_1005Metric, F.Cu at (313.6, 106.2)
- added C56: 10uF, Capacitor_SMD:C_0603_1608Metric, F.Cu at (308.2, 102.6)
- added C63: 1uF, Capacitor_SMD:C_0402_1005Metric, F.Cu at (313.6, 102.3)
- added C64: 10uF, Capacitor_SMD:C_0603_1608Metric, F.Cu at (308.2, 105.1)
- added C65: 10uF, Capacitor_SMD:C_0603_1608Metric, F.Cu at (308.2, 107.6)
- added FB10: FerriteBead, Inductor_SMD:L_0603_1608Metric, F.Cu at (308.2, 120.1)
- added FB3: FerriteBead, Inductor_SMD:L_0603_1608Metric, F.Cu at (314.2, 110.5)
- added FB4: FerriteBead, Inductor_SMD:L_0603_1608Metric, F.Cu at (314.2, 113.0)
- added FB5: FerriteBead, Inductor_SMD:L_0603_1608Metric, F.Cu at (314.2, 117.5)
- added FB6: FerriteBead, Inductor_SMD:L_0603_1608Metric, F.Cu at (314.2, 120.0)
- added FB7: FerriteBead, Inductor_SMD:L_0603_1608Metric, F.Cu at (308.2, 112.6)
- added FB8: FerriteBead, Inductor_SMD:L_0603_1608Metric, F.Cu at (308.2, 115.1)
- added FB9: FerriteBead, Inductor_SMD:L_0603_1608Metric, F.Cu at (308.2, 117.6)
- C100, C52, C53, C54, C55, C66, C67, C68, C69, C70, C71, C72, C73, C74, C75, C76, C83, C85, C86, C87, C88, C89, C90, C91, C92, C93, C94, C95, C96, C97, C98, C99: value 100nF -> 0.1uF
- C13, C14, C15, C16, C32, C33, C34, C35: value 0.1uF -> 1uF
- R20, R21: value 4.7k -> 0
- moved R37 356.4 mm to (109.8, 341.0)
Connections:
- C13 pad 2: +1V8 -> /LHC_CLK/+VDD
- C14 pad 2: +1V8 -> /LHC_CLK/+VDD
- C15 pad 2: +1V8 -> /LHC_CLK/+VDD
- C17 pad 2: +3V3 -> Net-(U1-VDDO0)
- C18 pad 2: +3V3 -> Net-(U1-VDDO0)
- C19 pad 2: +3V3 -> Net-(U1-VDDO0)
- C20 pad 2: +3V3 -> Net-(U1-VDDO0)
- C21 pad 2: +3V3 -> Net-(U1-VDDO0)
- C22 pad 2: +3V3 -> Net-(U1-VDDO0)
- C23 pad 2: +3V3 -> Net-(U1-VDDO0)
- C24 pad 2: +3V3 -> Net-(U1-VDDO0)
- C25 pad 2: +3V3 -> Net-(U1-VDDO0)
- C32 pad 2: +1V8 -> /LHC_CLK_HQ/+VDD
- C33 pad 2: +1V8 -> /LHC_CLK_HQ/+VDD
- C34 pad 2: +1V8 -> /LHC_CLK_HQ/+VDD
- C36 pad 2: +3V3 -> Net-(U2-VDDO0)
- C37 pad 2: +3V3 -> Net-(U2-VDDO0)
- C38 pad 2: +3V3 -> Net-(U2-VDDO0)
- C39 pad 2: +3V3 -> Net-(U2-VDDO0)
- C40 pad 2: +3V3 -> Net-(U2-VDDO0)
- C41 pad 2: +3V3 -> Net-(U2-VDDO0)
- C42 pad 2: +3V3 -> Net-(U2-VDDO0)
- C43 pad 2: +3V3 -> Net-(U2-VDDO0)
- C44 pad 2: +3V3 -> Net-(U2-VDDO0)
- C45 pad 2: +3V3 -> /SFP+/VccT1
- C46 pad 2: +3V3 -> /SFP+/VccR1
- C47 pad 2: +3V3 -> /SFP+/VccT2
- C48 pad 2: +3V3 -> /SFP+/VccR2
- C51 pad 1: +1V8 -> (no net)
- C51 pad 2: GND -> (no net)
- FB2 pad 1: +3V3 -> +1V8
- FB2 pad 2: /LHC_CLK_HQ/+VDDA -> /LHC_CLK_HQ/+VDD
- J6 pad 15: +3V3 -> /SFP+/VccR1
- J6 pad 16: +3V3 -> /SFP+/VccT1
- J6 pad CAGE: unconnected-(J6-PadCAGE) -> GNDPWR
- J7 pad 15: +3V3 -> /SFP+/VccR2
- J7 pad 16: +3V3 -> /SFP+/VccT2
- J7 pad 4: /LHC_CLK/SC_PLL.SDA -> unconnected-(J7-SDA-Pad4)
- J7 pad 6: /SFP+/SC_SFP+_2.MOD_ABS_2 -> /LHC_CLK/SC_PLL.SDA
- J7 pad CAGE: unconnected-(J7-PadCAGE) -> GNDPWR
- NT1 pad 1: Net-(U5-SENSE) -> (no net)
- NT1 pad 2: +1V8 -> (no net)
- Q5 pad 2: Net-(J17-Pin_2) -> +3V3
- R6 pad 2: /SFP+/SC_SFP+_2.MOD_ABS_2 -> /LHC_CLK/SC_PLL.SDA
- U1 pad 22: +3V3 -> Net-(U1-VDDO0)
- U1 pad 26: +3V3 -> Net-(U1-VDDO0)
- U1 pad 29: +3V3 -> Net-(U1-VDDO0)
- U1 pad 32: +1V8 -> /LHC_CLK/+VDD
- U1 pad 33: +3V3 -> Net-(U1-VDDO0)
- U1 pad 36: +3V3 -> Net-(U1-VDDO0)
- U1 pad 40: +3V3 -> Net-(U1-VDDO0)
- U1 pad 43: +3V3 -> Net-(U1-VDDO0)
- U1 pad 46: +1V8 -> /LHC_CLK/+VDD
- U1 pad 49: +3V3 -> Net-(U1-VDDO0)
- U1 pad 52: +3V3 -> Net-(U1-VDDO0)
- U1 pad 57: +3V3 -> Net-(U1-VDDO0)
- U1 pad 60: +1V8 -> /LHC_CLK/+VDD
- U2 pad 22: +3V3 -> Net-(U2-VDDO0)
- U2 pad 26: +3V3 -> Net-(U2-VDDO0)
- U2 pad 29: +3V3 -> Net-(U2-VDDO0)
- U2 pad 32: +1V8 -> /LHC_CLK_HQ/+VDD
- U2 pad 33: +3V3 -> Net-(U2-VDDO0)
- U2 pad 36: +3V3 -> Net-(U2-VDDO0)
- U2 pad 40: +3V3 -> Net-(U2-VDDO0)
- U2 pad 43: +3V3 -> Net-(U2-VDDO0)
- U2 pad 46: +1V8 -> /LHC_CLK_HQ/+VDD
- U2 pad 49: +3V3 -> Net-(U2-VDDO0)
- U2 pad 52: +3V3 -> Net-(U2-VDDO0)
- U2 pad 57: +3V3 -> Net-(U2-VDDO0)
- U2 pad 60: +1V8 -> /LHC_CLK_HQ/+VDD
- U3 pad 21: /LHC_CLK/SC_PLL.INTR -> /LHC_CLK/SC_PLL.FINC
- U3 pad 22: /LHC_CLK/SC_PLL.LOL -> /LHC_CLK/SC_PLL.FDEC
- U3 pad 24: /LHC_CLK_HQ/SC_PLL.RST -> /LHC_CLK/SC_PLL.INTR
- U3 pad 25: /LHC_CLK_HQ/SC_PLL.OE -> /LHC_CLK/SC_PLL.LOL
- U3 pad 26: /LHC_CLK_HQ/SC_PLL.INTR -> /LHC_CLK_HQ/SC_PLL.RST
- U3 pad 27: /LHC_CLK_HQ/SC_PLL.LOL -> /LHC_CLK_HQ/SC_PLL.OE
- U3 pad 29: unconnected-(U3-GPIO22-Pad29) -> /LHC_CLK_HQ/SC_PLL.FINC
- U3 pad 31: unconnected-(U3-GPIO26_ADC0-Pad31) -> /LHC_CLK_HQ/SC_PLL.FDEC
- U3 pad 32: unconnected-(U3-GPIO27_ADC1-Pad32) -> /LHC_CLK/SC_PLL.INTR
- U3 pad 34: unconnected-(U3-GPIO28_ADC2-Pad34) -> /LHC_CLK/SC_PLL.LOL
Routing:
- net +1V8: track 4.37 -> 0.00 mm, vias 1 -> 0
- net /LHC_CLK_HQ/+VDD: track 0.00 -> 2.19 mm, vias 0 -> 1
- net /LHC_CLK/+VDD: track 0.00 -> 2.19 mm
