File: atca-simple-loopback-hub.kicad_pcb (KiCad board)
At the start: 8 copper layers, 280 x 322.2 mm, 196 parts, among them J1 0826-1X4T-HS-F, J10 Conn_Coaxial, J11 Conn_Coaxial, J12 Conn_Coaxial, J13 Conn_Coaxial, J14 Conn_01x03_Male, J16 TE 2007262-1, J2 0826-1X4T-HS-F, J20 TE_64690XX-1_J20, J21 TE_64690XX-1_J21, J22 TE_64690XX-1_J22, J23 TE_64690XX-1_J23, J24 TE_64690XX-1_J24, J3 ESD_strip_bottom, J4 Conn_Coaxial, J5 Conn_Coaxial, J6 SFP+, J7 SFP+, J8 Conn_Coaxial, J9 Conn_Coaxial, K1 Key_K1_K2_TE_1-1469373-1, K2 Key_K1_K2_TE_1-1469373-1, P10 1766500-1, Q5 DMG2305UX, U1 Si5395, U2 Si5395, U3 Pico, U4 PIM400KZ, U5 ADM7172, X1 CX3225SB, X2 CX3225SB

Commit message: added loop between plls and monitoring sma at the second stage pll
Parts:
- removed NT1: Net-Tie_2, NetTie:NetTie-2_SMD_Pad0.5mm
- added C104: 0.1uF, Capacitor_SMD:C_0402_1005Metric, F.Cu at (289.0, 204.3)
- added C105: 0.1uF, Capacitor_SMD:C_0402_1005Metric, F.Cu at (289.0, 203.3)
- added C106: 0.1uF, Capacitor_SMD:C_0402_1005Metric, F.Cu at (289.0, 205.3)
- added R36: 50, Resistor_SMD:R_0402_1005Metric, F.Cu at (291.0, 203.8)
- added R38: 50, Resistor_SMD:R_0402_1005Metric, F.Cu at (291.0, 204.8)
- moved C63 217.0 mm to (98.2, 76.0), turned to -90 degrees
- moved C101 211.4 mm to (104.0, 77.0), turned to -90 degrees
- moved R20 177.7 mm to (142.5, 129.0)
- moved C56 171.2 mm to (143.0, 147.5)
- moved C102 170.4 mm to (143.0, 152.0)
- moved R21 168.9 mm to (142.5, 145.5)
- moved FB9 168.2 mm to (143.0, 149.0), turned to 180 degrees
- moved C65 168.0 mm to (143.0, 138.0)
- moved FB10 168.0 mm to (143.0, 150.5), turned to 180 degrees
- moved C64 167.6 mm to (143.0, 133.5)
- moved FB7 166.7 mm to (143.0, 135.0), turned to 180 degrees
- moved FB8 166.6 mm to (143.0, 136.5), turned to 180 degrees
- moved C103 66.8 mm to (301.8, 172.0)
- moved FB3 62.1 mm to (311.8, 172.5)
- moved FB4 59.8 mm to (304.5, 172.0)
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Connections:
- C51 pad 1: (no net) -> +1V8
- C51 pad 2: (no net) -> GND
- J6 pad 4: /ATCA_Z1/SC_PIM.SDA -> unconnected-(J6-SDA-Pad4)
- J6 pad 5: /ATCA_Z1/SC_PIM.SCL -> unconnected-(J6-SCL-Pad5)
- J6 pad 6: /SFP+/SC_SFP+_1.MOD_ABS_1 -> /ATCA_Z1/SC_PIM.SCL
- J7 pad 5: /LHC_CLK/SC_PLL.SCL -> unconnected-(J7-SCL-Pad5)
- R1 pad 2: /SFP+/SC_SFP+_1.MOD_ABS_1 -> /ATCA_Z1/SC_PIM.SCL
- U1 pad 1: unconnected-(U1-IN1-Pad1) -> /LHC_CLK/IN1_P
- U1 pad 11: /LHC_CLK/SC_PLL.OE -> /LHC_CLK/SC_PLL.RST
- U1 pad 2: unconnected-(U1-IN1b-Pad2) -> /LHC_CLK/IN1_N
- U1 pad 6: /LHC_CLK/SC_PLL.RST -> unconnected-(U1-~{RST}-Pad6)
- U2 pad 55: /Z2_FI11.LHC_CLK_HQ_N -> /LHC_CLK/CLK_intern.N
- U2 pad 56: /Z2_FI11.LHC_CLK_HQ_P -> /LHC_CLK/CLK_intern.P
- U3 pad 20: /LHC_CLK/SC_PLL.OE -> /LHC_CLK/SC_PLL.RST
Routing:
- net GND: track 2.12 -> 13.0 mm, vias 2 -> 3
- net /Z2_FI1.TCDS2_N: track 0.00 -> 8.85 mm, vias 0 -> 1
- net /LHC_CLK/IN1_N: track 0.00 -> 7.40 mm
- net /LHC_CLK/IN1_P: track 0.00 -> 7.39 mm
- net /LHC_CLK/CLK_intern.N: track 0.00 -> 5.25 mm
- net /LHC_CLK/CLK_intern.P: track 0.00 -> 5.08 mm
- net Net-(C104-Pad2): track 0.00 -> 2.41 mm
- net /Z2_FI11.LHC_CLK_HQ_P: track 11.9 -> 10.1 mm
- net /Z2_FI11.LHC_CLK_HQ_N: track 11.2 -> 9.36 mm

Commit message: routing z2
Parts:
- added J15: Conn_Coaxial, Connector_Coaxial:MMCX_Molex_73415-1471_Vertical, F.Cu at (291.7, 165.7)
- added J17: Conn_Coaxial, Connector_Coaxial:MMCX_Molex_73415-1471_Vertical, F.Cu at (291.7, 171.6)
- added NT1: Net-Tie_2, NetTie:NetTie-2_SMD_Pad0.5mm, F.Cu at (278.0, 227.1)
- moved C103 222.3 mm to (102.0, 74.5)
- moved J12 125.7 mm to (255.4, 270.4)
- moved J13 125.7 mm to (255.4, 260.8)
- moved FB5 69.9 mm to (292.2, 244.6)
- moved FB6 53.8 mm to (306.0, 232.8), turned to -90 degrees
- moved FB4 49.7 mm to (280.6, 215.5)
- moved FB3 48.7 mm to (292.5, 217.2)
- moved FB2 11.0 mm to (290.2, 233.8)
- moved C3 10.1 mm to (342.5, 255.2)
- moved C6 10.1 mm to (342.5, 251.8)
- moved C4 10.0 mm to (342.5, 254.2)
- moved C5 10.0 mm to (342.5, 252.8)
- moved R20 1.46 mm to (142.5, 130.5)
- moved R5 1.46 mm to (142.5, 129.5)
- moved C102 0.50 mm to (143.0, 152.5)
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Connections:
- net /LHC_CLK/CLK_intern.N renamed /LHC_CLK/CLK_Intern_I.N
- net /LHC_CLK/CLK_intern.P renamed /LHC_CLK/CLK_Intern_I.P
- net /LHC_CLK/SC_PLL.SCL renamed /LHC_CLK_HQ/SC_PLL.SCL
- net /LHC_CLK/SC_PLL.SDA renamed /LHC_CLK_HQ/SC_PLL.SDA
- J6 pad 6: /ATCA_Z1/SC_PIM.SCL -> /ATCA_Z1/SC_PIM.SDA
- R1 pad 2: /ATCA_Z1/SC_PIM.SCL -> /ATCA_Z1/SC_PIM.SDA
- U1 pad 11: /LHC_CLK/SC_PLL.RST -> /LHC_CLK/SC_PLL.OE
- U1 pad 55: /Z2_FI11.LHC_CLK_N -> /LHC_CLK/CLK_Intern_O.N
- U1 pad 56: /Z2_FI11.LHC_CLK_P -> /LHC_CLK/CLK_Intern_O.P
- U1 pad 6: unconnected-(U1-~{RST}-Pad6) -> /LHC_CLK/SC_PLL.RST
- U3 pad 20: /LHC_CLK/SC_PLL.RST -> /LHC_CLK/SC_PLL.OE
Routing:
- net /Z2_FI3.LHC_CLK_HQ_P: track 67.7 -> 6.29 mm
- net /Z2_FI3.LHC_CLK_HQ_N: track 67.3 -> 6.12 mm
- net /Z2_FI2.LHC_CLK_HQ_P: track 72.6 -> 17.4 mm
- net /Z2_FI2.LHC_CLK_HQ_N: track 71.9 -> 17.0 mm
- net /J22/10GbE_RX_N: track 14.5 -> 27.3 mm, vias 0 -> 1
- net /Z2_FI3.10GbE_TX_P: track 0.00 -> 12.8 mm
- net /Z2_FI3.10GbE_TX_N: track 0.00 -> 12.8 mm
- net /J22/LVDS_RX_N: track 6.64 -> 19.2 mm
- net /Z2_FI3.TCDS2_TX_P: track 0.00 -> 12.2 mm
- net /Z2_FI3.TCDS2_TX_N: track 0.00 -> 12.2 mm
- net /J22/10GbE_RX_P: track 16.0 -> 28.0 mm, vias 0 -> 1
- net /Z2_FI3.10GbE_RX_P: track 0.00 -> 12.0 mm
- net /Z2_FI3.10GbE_RX_N: track 0.00 -> 12.0 mm
- net /Z2_FI3.TCDS2_RX_P: track 0.00 -> 11.6 mm
- net /Z2_FI3.TCDS2_RX_N: track 0.00 -> 11.6 mm
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
Commit message: routing eth
Parts:
- moved J13 18.3 mm to (264.7, 245.0)
- moved J12 18.3 mm to (264.7, 254.7)
Routing:
- net /Z2_BI8.A_P: track 0.00 -> 260.7 mm, vias 0 -> 1
- net /Z2_BI8.B_P: track 0.00 -> 260.2 mm, vias 0 -> 1
- net /Z2_BI8.A_N: track 0.00 -> 260.2 mm, vias 0 -> 1
- net /Z2_BI8.B_N: track 0.00 -> 259.7 mm, vias 0 -> 1
- net /Z2_BI8.C_P: track 0.00 -> 254.4 mm
- net /Z2_BI8.C_N: track 0.00 -> 254.0 mm
- net /Z2_BI7.C_P: track 0.00 -> 249.4 mm, vias 0 -> 2
- net /Z2_BI7.C_N: track 0.00 -> 248.6 mm, vias 0 -> 2
- net /Z2_BI8.D_P: track 0.00 -> 247.1 mm, vias 0 -> 1
- net /Z2_BI8.D_N: track 0.00 -> 246.7 mm, vias 0 -> 1
- net /Z2_BI7.A_P: track 0.00 -> 233.4 mm, vias 0 -> 1
- net /Z2_BI7.A_N: track 0.00 -> 233.0 mm, vias 0 -> 1
- net /Z2_BI6.A_P: track 0.00 -> 232.5 mm, vias 0 -> 1
- net /Z2_BI6.A_N: track 0.00 -> 232.2 mm, vias 0 -> 1
- net /Z2_BI6.B_P: track 0.00 -> 230.6 mm, vias 0 -> 1
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