File: sch/mech.kicad_sch (KiCad schematic)
At the start: 13 parts, among them J12 Conn_01x03_Male, J3 ESD_strip_bottom, K1 Key_K1_K2_TE_1-1469373-1, K2 Key_K1_K2_TE_1-1469373-1

Commit message: all signals routed
Connections:
- net +3V3_STBY renamed +3V3
Changed lines of the file:
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@@
 	(wire
 		(pts
-			(xy 118.11 138.43) (xy 115.57 138.43)
+			(xy 123.19 138.43) (xy 115.57 138.43)
 		)
 		(stroke
@@
 		)
 	)
-	(global_label "FP_HANDLE"
+	(hierarchical_label "FP_HANDLE"
 		(shape output)
-		(at 118.11 138.43 0)
+		(at 123.19 138.43 0)
+		(fields_autoplaced yes)
 		(effects
 			(font
@@
 			)
 			(justify left)
-		)
-		(property "Intersheetrefs" "${INTERSHEET_REFS}"
-			(at 118.11 138.43 0)
-			(effects
-				(font
-					(size 1.27 1.27)
-				)
-				(hide yes)
-			)
 		)
 	)
@@
 	)
 	(symbol
-		(lib_id "KIT_Power:+3V3_STBY")
-		(at 115.57 125.73 0)
-		(unit 1)
-		(exclude_from_sim no)
-		(in_bom yes)
-		(on_board yes)
-		(dnp no)
-		(property "Reference" "#PWR?"
-			(at 115.57 129.54 0)
-			(effects
-				(font
-					(size 1.27 1.27)
-				)
-				(hide yes)
-			)
-		)
-		(property "Value" "+3V3_STBY"
-			(at 115.951 121.3358 0)
-			(effects
-				(font
-					(size 1.27 1.27)
-				)
-			)
-		)
-		(property "Footprint" ""
-			(at 115.57 125.73 0)
-			(effects
-				(font
-					(size 1.27 1.27)
-				)
-				(hide yes)
-			)
-		)
-		(property "Datasheet" ""
-			(at 115.57 125.73 0)
-			(effects
-				(font
-					(size 1.27 1.27)
-				)
-				(hide yes)
-			)
-		)
-		(property "Description" ""
-			(at 115.57 125.73 0)
-			(effects
-				(font
-					(size 1.27 1.27)
-				)
-				(hide yes)
-			)
-		)
-		(pin "1"
-		)
-		(instances
-			(project "atca_zynqmp"
-				(path "/379f62ac-1342-42f2-a04b-e91c669e9899"
-					(reference "#PWR?")
-					(unit 1)
-				)
-				(path "/379f62ac-1342-42f2-a04b-e91c669e9899/00000000-0000-0000-0000-00005d1343c8"
-					(reference "#PWR?")
-					(unit 1)
-				)
-			)
-			(project "atca-simple-loopback-hub"
-				(path "/b1bf14e0-f6d2-45a7-b67f-6500a354b7ad/f77876dd-ebdc-4e20-8c96-1773c09aca35"
-					(reference "#PWR0112")
-					(unit 1)
-				)
-			)
-		)
-	)
-	(symbol
 		(lib_id "project:Key_K1_K2_TE_1-1469373-1")
 		(at 175.26 57.15 0)
@@
 					(unit 1)
 				)
+			)
+		)
+	)
+	(symbol
+		(lib_id "power:+3V3")
+		(at 115.57 125.73 0)
+		(unit 1)
+		(exclude_from_sim no)
+		(in_bom yes)
+		(on_board yes)
+		(dnp no)
+		(fields_autoplaced yes)
+		(property "Reference" "#PWR0112"
+			(at 115.57 129.54 0)
+			(effects
+				(font
+					(size 1.27 1.27)
+				)
+				(hide yes)
+			)
+		)
+		(property "Value" "+3V3"
+			(at 115.57 120.65 0)
+			(effects
+				(font
+					(size 1.27 1.27)
+				)
+			)
+		)
+		(property "Footprint" ""
+			(at 115.57 125.73 0)
+			(effects
+				(font
+					(size 1.27 1.27)
+				)
+				(hide yes)
+			)
+		)
+		(property "Datasheet" ""
+			(at 115.57 125.73 0)
+			(effects
+				(font
+					(size 1.27 1.27)
+				)
+				(hide yes)
+			)
+		)
+		(property "Description" ""
+			(at 115.57 125.73 0)
+			(effects
+				(font
+					(size 1.27 1.27)
+				)
+				(hide yes)
+			)
+		)
+		(pin "1"
+		)
+		(instances
+			(project "atca-simple-loopback-hub"
+				(path "/b1bf14e0-f6d2-45a7-b67f-6500a354b7ad/f77876dd-ebdc-4e20-8c96-1773c09aca35"
+					(reference "#PWR0112")
+					(unit 1)
+				)

Commit message: fully routed board
Parts:
- added H6, H7: MountingHole, project:NPTH_2.7_7_Keepout, symbol project:MountingHole
Other:
- moved on the sheet: H3, H4, H5
Changed lines of the file:
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@@
+	)
+	(symbol
+		(lib_id "project:MountingHole")
+		(at 144.78 101.6 0)
+		(unit 1)
+		(exclude_from_sim no)
+		(in_bom yes)
+		(on_board yes)
+		(dnp no)
+		(fields_autoplaced yes)
+		(property "Reference" "H7"
+			(at 147.32 100.3299 0)
+			(effects
+				(font
+					(size 1.27 1.27)
+				)
+				(justify left)
+			)
+		)
+		(property "Value" "MountingHole"
+			(at 147.32 102.8699 0)
+			(effects
+				(font
+					(size 1.27 1.27)
+				)
+				(justify left)
+			)
+		)
+		(property "Footprint" "project:NPTH_2.7_7_Keepout"
+			(at 144.78 101.6 0)
+			(effects
+				(font
+					(size 1.27 1.27)
+				)
+				(hide yes)
+			)
+		)
+		(property "Datasheet" "~"
+			(at 144.78 101.6 0)
+			(effects
+				(font
+					(size 1.27 1.27)
+				)
+				(hide yes)
+			)
+		)
+		(property "Description" ""
+			(at 144.78 101.6 0)
+			(effects
+				(font
+					(size 1.27 1.27)
+				)
+				(hide yes)
+			)
+		)
+		(property "stock" "PCB"
+			(at 144.78 101.6 0)
+			(effects
+				(font
+					(size 1.27 1.27)
+				)
+				(hide yes)
+			)
+		)
+		(instances
+			(project "atca-simple-loopback-hub"
+				(path "/b1bf14e0-f6d2-45a7-b67f-6500a354b7ad/f77876dd-ebdc-4e20-8c96-1773c09aca35"
+					(reference "H7")
+					(unit 1)
+				)
+			)
+		)
 	)
 	(symbol
@@
 	(symbol
 		(lib_id "project:MountingHole")
-		(at 146.05 64.77 0)
+		(at 163.83 64.77 0)
 		(unit 1)
 		(exclude_from_sim no)
@@
 		(fields_autoplaced yes)
 		(property "Reference" "H3"
-			(at 148.59 63.4999 0)
+			(at 166.37 63.4999 0)
 			(effects
 				(font
@@
 		)
 		(property "Value" "MountingHole"
-			(at 148.59 66.0399 0)
+			(at 166.37 66.0399 0)
 			(effects
 				(font
@@
 		)
 		(property "Footprint" "project:NPTH_2.7_7_Keepout"
-			(at 146.05 64.77 0)
+			(at 163.83 64.77 0)
 			(effects
 				(font
@@
 		)
 		(property "Datasheet" "~"
-			(at 146.05 64.77 0)
-			(effects
-				(font
-					(size 1.27 1.27)
-				)
-				(hide yes)
-			)
-		)
-		(property "Description" ""
-			(at 146.05 64.77 0)
+			(at 163.83 64.77 0)
+			(effects
+				(font
+					(size 1.27 1.27)
+				)
+				(hide yes)
+			)
+		)
+		(property "Description" ""
+			(at 163.83 64.77 0)
 			(effects
 				(font
@@
 		)
 		(property "stock" "PCB"
-			(at 146.05 64.77 0)
+			(at 163.83 64.77 0)
 			(effects
 				(font
@@
 	(symbol
 		(lib_id "project:MountingHole")
-		(at 146.05 97.79 0)
+		(at 163.83 95.25 0)
 		(unit 1)
 		(exclude_from_sim no)
@@
 		(fields_autoplaced yes)
 		(property "Reference" "H4"
-			(at 148.59 96.5199 0)
+			(at 166.37 93.9799 0)
 			(effects
 				(font
@@
 		)
 		(property "Value" "MountingHole"
-			(at 148.59 99.0599 0)
+			(at 166.37 96.5199 0)
 			(effects
 				(font
@@
 		)
 		(property "Footprint" "project:NPTH_2.7_7_Keepout"
-			(at 146.05 97.79 0)
+			(at 163.83 95.25 0)
 			(effects
 				(font
@@
 		)
 		(property "Datasheet" "~"
-			(at 146.05 97.79 0)
-			(effects
-				(font
-					(size 1.27 1.27)
-				)
-				(hide yes)
-			)
-		)
-		(property "Description" ""
-			(at 146.05 97.79 0)
+			(at 163.83 95.25 0)
+			(effects
+				(font
+					(size 1.27 1.27)
+				)
+				(hide yes)
+			)
+		)
+		(property "Description" ""
+			(at 163.83 95.25 0)
 			(effects
 				(font
@@
 		)
 		(property "stock" "PCB"
-			(at 146.05 97.79 0)
+			(at 163.83 95.25 0)
 			(effects
 				(font
@@
 	(symbol
 		(lib_id "project:MountingHole")
-		(at 166.37 97.79 0)
+		(at 163.83 101.6 0)
 		(unit 1)
 		(exclude_from_sim no)
@@
 		(fields_autoplaced yes)
 		(property "Reference" "H5"
-			(at 168.91 96.5199 0)
+			(at 166.37 100.3299 0)
 			(effects
 				(font
@@
 		)
 		(property "Value" "MountingHole"
-			(at 168.91 99.0599 0)
+			(at 166.37 102.8699 0)
 			(effects
 				(font
@@
 		)
 		(property "Footprint" "project:NPTH_2.7_7_Keepout"
-			(at 166.37 97.79 0)
+			(at 163.83 101.6 0)
 			(effects
 				(font
@@
 		)
 		(property "Datasheet" "~"
-			(at 166.37 97.79 0)
-			(effects
-				(font
-					(size 1.27 1.27)
-				)
-				(hide yes)
-			)
-		)
-		(property "Description" ""
-			(at 166.37 97.79 0)
+			(at 163.83 101.6 0)
+			(effects
+				(font
+					(size 1.27 1.27)
+				)
+				(hide yes)
+			)
+		)
+		(property "Description" ""
+			(at 163.83 101.6 0)
 			(effects
 				(font
@@
 		)
 		(property "stock" "PCB"
-			(at 166.37 97.79 0)
+			(at 163.83 101.6 0)
 			(effects
 				(font
@@
 					(unit 1)
 				)
+			)
+		)
+	)
+	(symbol
+		(lib_id "project:MountingHole")
+		(at 144.78 64.77 0)
+		(unit 1)
+		(exclude_from_sim no)
+		(in_bom yes)
+		(on_board yes)
+		(dnp no)
+		(fields_autoplaced yes)
+		(property "Reference" "H6"
+			(at 147.32 63.4999 0)
+			(effects
+				(font
+					(size 1.27 1.27)
+				)
+				(justify left)
+			)
+		)
+		(property "Value" "MountingHole"
+			(at 147.32 66.0399 0)
+			(effects
+				(font
+					(size 1.27 1.27)
+				)
+				(justify left)
+			)
+		)
+		(property "Footprint" "project:NPTH_2.7_7_Keepout"
+			(at 144.78 64.77 0)
+			(effects
+				(font
+					(size 1.27 1.27)
+				)
+				(hide yes)
+			)
+		)
+		(property "Datasheet" "~"
+			(at 144.78 64.77 0)
+			(effects
+				(font
+					(size 1.27 1.27)
+				)
+				(hide yes)
+			)
+		)
+		(property "Description" ""
+			(at 144.78 64.77 0)
+			(effects
+				(font
+					(size 1.27 1.27)
+				)
+				(hide yes)
+			)
+		)
+		(property "stock" "PCB"
+			(at 144.78 64.77 0)
+			(effects
+				(font
+					(size 1.27 1.27)
+				)
+				(hide yes)
+			)
+		)
+		(instances
+			(project "atca-simple-loopback-hub"
+				(path "/b1bf14e0-f6d2-45a7-b67f-6500a354b7ad/f77876dd-ebdc-4e20-8c96-1773c09aca35"
+					(reference "H6")
+					(unit 1)
+				)
