File: sch/ATCA_Z1.kicad_sch (KiCad schematic)
At the start: 26 parts, among them P10 1766500-1, U4 PIM400KZ

Commit message: v1.0 as fabricated
Parts:
- added C107: 100uF, Capacitor_SMD:CP_Elec_18x22, symbol Device:C_Polarized
- added J18: Conn_01x02_Pin, Connector_Wago:Wago_734-132_1x02_P3.50mm_Vertical, symbol Connector:Conn_01x02_Pin
Connections:
- net BUS_N: now also C107.2, J18.2 (Pin_2)
- net BUS_P: now also C107.1, J18.1 (Pin_1)
- net R_HLDP: now reaches R7.2, U4.16 (TRIM_HLDP)
Other:
- moved on the sheet: C82, C84, R7
