File: sch/LHC_CLK.kicad_sch (KiCad schematic)
At the start: 38 parts, among them U1 Si5395, X1 CX3225SB

Commit message: routing PLLs
Connections:
- net Z2_FI1.LHC_CLK_N: now also U1.21 (OUT0A); no longer U1.20 (OUT0Ab)
- net Z2_FI1.LHC_CLK_P: now also U1.20 (OUT0Ab); no longer U1.21 (OUT0A)
- net Z2_FI10.LHC_CLK_N: now also U1.54 (OUT8); no longer U1.53 (OUT8b)
- net Z2_FI10.LHC_CLK_P: now also U1.53 (OUT8b); no longer U1.54 (OUT8)
- net Z2_FI2.LHC_CLK_N: now also U1.24 (OUT0); no longer U1.23 (OUT0b)
- net Z2_FI2.LHC_CLK_P: now also U1.23 (OUT0b); no longer U1.24 (OUT0)
- net Z2_FI3.LHC_CLK_N: now also U1.28 (OUT1); no longer U1.27 (OUT1b)
- net Z2_FI3.LHC_CLK_P: now also U1.27 (OUT1b); no longer U1.28 (OUT1)
- net Z2_FI4.LHC_CLK_N: now also U1.31 (OUT2); no longer U1.30 (OUT2b)
- net Z2_FI4.LHC_CLK_P: now also U1.30 (OUT2b); no longer U1.31 (OUT2)
- net Z2_FI5.LHC_CLK_N: now also U1.35 (OUT3); no longer U1.34 (OUT3b)
- net Z2_FI5.LHC_CLK_P: now also U1.34 (OUT3b); no longer U1.35 (OUT3)
- net Z2_FI6.LHC_CLK_N: now also U1.38 (OUT4); no longer U1.37 (OUT4b)
- net Z2_FI6.LHC_CLK_P: now also U1.37 (OUT4b); no longer U1.38 (OUT4)
- net Z2_FI7.LHC_CLK_N: now also U1.42 (OUT5); no longer U1.41 (OUT5b)
- net Z2_FI7.LHC_CLK_P: now also U1.41 (OUT5b); no longer U1.42 (OUT5)
- net Z2_FI8.LHC_CLK_N: now also U1.45 (OUT6); no longer U1.44 (OUT6b)
- net Z2_FI8.LHC_CLK_P: now also U1.44 (OUT6b); no longer U1.45 (OUT6)
- net Z2_FI9.LHC_CLK_N: now also U1.51 (OUT7); no longer U1.50 (OUT7b)
- net Z2_FI9.LHC_CLK_P: now also U1.50 (OUT7b); no longer U1.51 (OUT7)
Changed lines of the file:
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@@
+	)
+	(junction
+		(at 200.66 26.67)
+		(diameter 0)
+		(color 0 0 0 0)
+	)
+	(junction
+		(at 147.32 35.56)
+		(diameter 0)
+		(color 0 0 0 0)
+	)
+	(junction
+		(at 180.34 35.56)
+		(diameter 0)
+		(color 0 0 0 0)
+	)
+	(junction
+		(at 149.86 19.05)
+		(diameter 0)
+		(color 0 0 0 0)
+	)
+	(junction
+		(at 234.95 26.67)
+		(diameter 0)
+		(color 0 0 0 0)
+	)
+	(junction
+		(at 189.23 26.67)
+		(diameter 0)
+		(color 0 0 0 0)
+	)
+	(junction
+		(at 45.72 128.27)
+		(diameter 0)
+		(color 0 0 0 0)
+	)
+	(junction
+		(at 200.66 19.05)
+		(diameter 0)
+		(color 0 0 0 0)
+	)
+	(junction
+		(at 212.09 26.67)
+		(diameter 0)
+		(color 0 0 0 0)
+	)
+	(junction
+		(at 116.84 88.9)
+		(diameter 0)
+		(color 0 0 0 0)
+	)
+	(junction
+		(at 67.31 67.31)
+		(diameter 0)
+		(color 0 0 0 0)
+	)
+	(junction
+		(at 59.69 144.78)
+		(diameter 0)
+		(color 0 0 0 0)
+	)
+	(junction
+		(at 189.23 19.05)
+		(diameter 0)
+		(color 0 0 0 0)
+	)
+	(junction
+		(at 127 101.6)
+		(diameter 0)
+		(color 0 0 0 0)
+	)
+	(junction
+		(at 96.52 19.05)
+		(diameter 0)
+		(color 0 0 0 0)
+	)
+	(junction
+		(at 149.86 35.56)
+		(diameter 0)
+		(color 0 0 0 0)
+	)
+	(junction
+		(at 172.72 35.56)
+		(diameter 0)
+		(color 0 0 0 0)
+	)
+	(junction
+		(at 59.69 111.76)
+		(diameter 0)
+		(color 0 0 0 0)
+	)
+	(junction
+		(at 67.31 100.33)
+		(diameter 0)
+		(color 0 0 0 0)
 	)
 	(junction
@@
 		(color 0 0 0 0)
 	)
-	(junction
-		(at 200.66 26.67)
-		(diameter 0)
-		(color 0 0 0 0)
-	)
-	(junction
-		(at 147.32 35.56)
-		(diameter 0)
-		(color 0 0 0 0)
-	)
-	(junction
-		(at 180.34 35.56)
-		(diameter 0)
-		(color 0 0 0 0)
-	)
-	(junction
-		(at 149.86 19.05)
-		(diameter 0)
-		(color 0 0 0 0)
-	)
-	(junction
-		(at 234.95 26.67)
-		(diameter 0)
-		(color 0 0 0 0)
-	)
-	(junction
-		(at 189.23 26.67)
-		(diameter 0)
-		(color 0 0 0 0)
-	)
-	(junction
-		(at 45.72 128.27)
-		(diameter 0)
-		(color 0 0 0 0)
-	)
-	(junction
-		(at 200.66 19.05)
-		(diameter 0)
-		(color 0 0 0 0)
-	)
-	(junction
-		(at 212.09 26.67)
-		(diameter 0)
-		(color 0 0 0 0)
-	)
-	(junction
-		(at 116.84 88.9)
-		(diameter 0)
-		(color 0 0 0 0)
-	)
-	(junction
-		(at 67.31 67.31)
-		(diameter 0)
-		(color 0 0 0 0)
-	)
-	(junction
-		(at 59.69 144.78)
-		(diameter 0)
-		(color 0 0 0 0)
-	)
-	(junction
-		(at 189.23 19.05)
-		(diameter 0)
-		(color 0 0 0 0)
-	)
-	(junction
-		(at 127 101.6)
-		(diameter 0)
-		(color 0 0 0 0)
-	)
-	(junction
-		(at 96.52 19.05)
-		(diameter 0)
-		(color 0 0 0 0)
-	)
-	(junction
-		(at 149.86 35.56)
-		(diameter 0)
-		(color 0 0 0 0)
-	)
-	(junction
-		(at 172.72 35.56)
-		(diameter 0)
-		(color 0 0 0 0)
-	)
-	(junction
-		(at 59.69 111.76)
-		(diameter 0)
-		(color 0 0 0 0)
-	)
-	(junction
-		(at 67.31 100.33)
-		(diameter 0)
-		(color 0 0 0 0)
-	)
 	(no_connect
 		(at 134.62 76.2)
@@
 	(wire
 		(pts
+			(xy 257.81 19.05) (xy 270.51 19.05)
+		)
+		(stroke
+			(width 0)
+			(type default)
+		)
+	)
+	(wire
+		(pts
 			(xy 62.23 144.78) (xy 62.23 129.54)
 		)
@@
 	(wire
 		(pts
-			(xy 257.81 19.05) (xy 270.51 19.05)
+			(xy 257.81 19.05) (xy 246.38 19.05)
 		)
 		(stroke
@@
 	(wire
 		(pts
-			(xy 246.38 19.05) (xy 257.81 19.05)
-		)
-		(stroke
-			(width 0)
-			(type default)
-		)
-	)
-	(wire
-		(pts
 			(xy 60.96 54.61) (xy 63.5 54.61)
 		)
@@
 			(width 0)
 			(type default)
+		)
+	)
+	(rectangle
+		(start 201.93 46.99)
+		(end 205.74 124.46)
+		(stroke
+			(width 0)
+			(type dash)
+		)
+		(fill
+			(type none)
 		)
 	)
@@
 		)
 	)
+	(text_box "P and N inverted"
+		(exclude_from_sim no)
+		(at 201.93 38.1 0)
+		(size 24.13 8.89)
+		(stroke
+			(width 0)
+			(type dash)
+		)
+		(fill
+			(type none)
+		)
+		(effects
+			(font
+				(size 1.27 1.27)
+				(bold yes)
+			)
+			(justify left top)
+		)
+	)
 	(text "48Mhz"
 		(exclude_from_sim no)
@@
 	)
 	(label "Z2_FI7.LHC_CLK_N"
-		(at 227.33 100.33 180)
+		(at 227.33 97.79 180)
 		(fields_autoplaced yes)
 		(effects
@@
 	)
 	(label "Z2_FI7.LHC_CLK_P"
-		(at 227.33 97.79 180)
+		(at 227.33 100.33 180)
 		(fields_autoplaced yes)
 		(effects
@@
 	)
 	(label "Z2_FI9.LHC_CLK_P"
-		(at 227.33 113.03 180)
+		(at 227.33 115.57 180)
 		(fields_autoplaced yes)
 		(effects
@@
 	)
 	(label "Z2_FI8.LHC_CLK_P"
-		(at 227.33 105.41 180)
+		(at 227.33 107.95 180)
 		(fields_autoplaced yes)
 		(effects
@@
 	)
 	(label "Z2_FI1.LHC_CLK_N"
-		(at 227.33 54.61 180)
+		(at 227.33 52.07 180)
 		(fields_autoplaced yes)
 		(effects
@@
 	)
 	(label "Z2_FI10.LHC_CLK_P"
-		(at 227.33 120.65 180)
+		(at 227.33 123.19 180)
 		(fields_autoplaced yes)
 		(effects
@@
 	)
 	(label "Z2_FI5.LHC_CLK_P"
-		(at 227.33 82.55 180)
+		(at 227.33 85.09 180)
 		(fields_autoplaced yes)
 		(effects
@@
 	)
 	(label "Z2_FI8.LHC_CLK_N"
-		(at 227.33 107.95 180)
+		(at 227.33 105.41 180)
 		(fields_autoplaced yes)
 		(effects
@@
 	)
 	(label "Z2_FI3.LHC_CLK_P"
-		(at 227.33 67.31 180)
+		(at 227.33 69.85 180)
 		(fields_autoplaced yes)
 		(effects
@@
 	)
 	(label "Z2_FI2.LHC_CLK_P"
-		(at 227.33 59.69 180)
+		(at 227.33 62.23 180)
 		(fields_autoplaced yes)
 		(effects
@@
 	)
 	(label "Z2_FI10.LHC_CLK_N"
-		(at 227.33 123.19 180)
+		(at 227.33 120.65 180)
 		(fields_autoplaced yes)
 		(effects
@@
 	)
 	(label "Z2_FI6.LHC_CLK_P"
-		(at 227.33 90.17 180)
+		(at 227.33 92.71 180)
 		(fields_autoplaced yes)
 		(effects
@@
 	)
 	(label "Z2_FI5.LHC_CLK_N"
-		(at 227.33 85.09 180)
+		(at 227.33 82.55 180)
 		(fields_autoplaced yes)
 		(effects
@@
 	)
 	(label "Z2_FI6.LHC_CLK_N"
-		(at 227.33 92.71 180)
+		(at 227.33 90.17 180)
 		(fields_autoplaced yes)
 		(effects
@@
 	)
 	(label "Z2_FI9.LHC_CLK_N"
-		(at 227.33 115.57 180)
+		(at 227.33 113.03 180)
 		(fields_autoplaced yes)
 		(effects
@@
 	)
 	(label "Z2_FI4.LHC_CLK_P"
+		(at 227.33 77.47 180)
+		(fields_autoplaced yes)
+		(effects
+			(font
+				(size 1.27 1.27)
+			)
+			(justify right bottom)
+		)
+	)
+	(label "Z2_FI1.LHC_CLK_P"
+		(at 227.33 54.61 180)
+		(fields_autoplaced yes)
+		(effects
+			(font
+				(size 1.27 1.27)
+			)
+			(justify right bottom)
+		)
+	)
+	(label "Z2_FI4.LHC_CLK_N"
 		(at 227.33 74.93 180)
 		(fields_autoplaced yes)
@@
 		)
 	)
-	(label "Z2_FI1.LHC_CLK_P"
-		(at 227.33 52.07 180)
-		(fields_autoplaced yes)
-		(effects
-			(font
-				(size 1.27 1.27)
-			)
-			(justify right bottom)
-		)
-	)
-	(label "Z2_FI4.LHC_CLK_N"
-		(at 227.33 77.47 180)
-		(fields_autoplaced yes)
-		(effects
-			(font
-				(size 1.27 1.27)
-			)
-			(justify right bottom)
-		)
-	)
 	(label "Z2_FI3.LHC_CLK_N"
-		(at 227.33 69.85 180)
+		(at 227.33 67.31 180)
 		(fields_autoplaced yes)
 		(effects
@@
 	)
 	(label "Z2_FI2.LHC_CLK_N"
-		(at 227.33 62.23 180)
-		(fields_autoplaced yes)
-		(effects
+		(at 227.33 59.69 180)
+		(fields_autoplaced yes)
+		(effects
