File: sch/LHC_CLK_HQ.kicad_sch (KiCad schematic)
At the start: 33 parts, among them U2 Si5395, X2 CX3225SB

Commit message: routing PLLs
Connections:
- net Z2_FI1.LHC_CLK_HQ_N: now also U2.21 (OUT0A); no longer U2.20 (OUT0Ab)
- net Z2_FI1.LHC_CLK_HQ_P: now also U2.20 (OUT0Ab); no longer U2.21 (OUT0A)
- net Z2_FI10.LHC_CLK_HQ_N: now also U2.54 (OUT8); no longer U2.53 (OUT8b)
- net Z2_FI10.LHC_CLK_HQ_P: now also U2.53 (OUT8b); no longer U2.54 (OUT8)
- net Z2_FI2.LHC_CLK_HQ_N: now also U2.24 (OUT0); no longer U2.23 (OUT0b)
- net Z2_FI2.LHC_CLK_HQ_P: now also U2.23 (OUT0b); no longer U2.24 (OUT0)
- net Z2_FI3.LHC_CLK_HQ_N: now also U2.28 (OUT1); no longer U2.27 (OUT1b)
- net Z2_FI3.LHC_CLK_HQ_P: now also U2.27 (OUT1b); no longer U2.28 (OUT1)
- net Z2_FI4.LHC_CLK_HQ_N: now also U2.31 (OUT2); no longer U2.30 (OUT2b)
- net Z2_FI4.LHC_CLK_HQ_P: now also U2.30 (OUT2b); no longer U2.31 (OUT2)
- net Z2_FI5.LHC_CLK_HQ_N: now also U2.35 (OUT3); no longer U2.34 (OUT3b)
- net Z2_FI5.LHC_CLK_HQ_P: now also U2.34 (OUT3b); no longer U2.35 (OUT3)
- net Z2_FI6.LHC_CLK_HQ_N: now also U2.38 (OUT4); no longer U2.37 (OUT4b)
- net Z2_FI6.LHC_CLK_HQ_P: now also U2.37 (OUT4b); no longer U2.38 (OUT4)
- net Z2_FI7.LHC_CLK_HQ_N: now also U2.42 (OUT5); no longer U2.41 (OUT5b)
- net Z2_FI7.LHC_CLK_HQ_P: now also U2.41 (OUT5b); no longer U2.42 (OUT5)
- net Z2_FI8.LHC_CLK_HQ_N: now also U2.45 (OUT6); no longer U2.44 (OUT6b)
- net Z2_FI8.LHC_CLK_HQ_P: now also U2.44 (OUT6b); no longer U2.45 (OUT6)
- net Z2_FI9.LHC_CLK_HQ_N: now also U2.51 (OUT7); no longer U2.50 (OUT7b)
- net Z2_FI9.LHC_CLK_HQ_P: now also U2.50 (OUT7b); no longer U2.51 (OUT7)
Changed lines of the file:
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@@
+		)
+	)
+	(rectangle
+		(start 199.39 46.99)
+		(end 203.2 124.46)
+		(stroke
+			(width 0)
+			(type dash)
+		)
+		(fill
+			(type none)
 		)
 	)
@@
 		)
 	)
+	(text_box "P and N inverted"
+		(exclude_from_sim no)
+		(at 199.39 38.1 0)
+		(size 24.13 8.89)
+		(stroke
+			(width 0)
+			(type dash)
+		)
+		(fill
+			(type none)
+		)
+		(effects
+			(font
+				(size 1.27 1.27)
+				(bold yes)
+			)
+			(justify left top)
+		)
+	)
 	(text "I2C Address = 8'b1101_001X, 8'hD2, 7'h69"
 		(exclude_from_sim no)
@@
 	)
 	(label "Z2_FI6.LHC_CLK_HQ_N"
-		(at 227.33 92.71 180)
+		(at 227.33 90.17 180)
 		(fields_autoplaced yes)
 		(effects
@@
 	)
 	(label "Z2_FI1.LHC_CLK_HQ_P"
-		(at 227.33 52.07 180)
+		(at 227.33 54.61 180)
 		(fields_autoplaced yes)
 		(effects
@@
 	)
 	(label "Z2_FI5.LHC_CLK_HQ_P"
-		(at 227.33 82.55 180)
+		(at 227.33 85.09 180)
 		(fields_autoplaced yes)
 		(effects
@@
 	)
 	(label "Z2_FI3.LHC_CLK_HQ_P"
-		(at 227.33 67.31 180)
+		(at 227.33 69.85 180)
 		(fields_autoplaced yes)
 		(effects
@@
 	)
 	(label "Z2_FI9.LHC_CLK_HQ_P"
-		(at 227.33 113.03 180)
+		(at 227.33 115.57 180)
 		(fields_autoplaced yes)
 		(effects
@@
 	)
 	(label "Z2_FI10.LHC_CLK_HQ_P"
-		(at 227.33 120.65 180)
+		(at 227.33 123.19 180)
 		(fields_autoplaced yes)
 		(effects
@@
 	)
 	(label "Z2_FI7.LHC_CLK_HQ_P"
-		(at 227.33 97.79 180)
+		(at 227.33 100.33 180)
 		(fields_autoplaced yes)
 		(effects
@@
 	)
 	(label "Z2_FI1.LHC_CLK_HQ_N"
-		(at 227.33 54.61 180)
+		(at 227.33 52.07 180)
 		(fields_autoplaced yes)
 		(effects
@@
 	)
 	(label "Z2_FI10.LHC_CLK_HQ_N"
-		(at 227.33 123.19 180)
+		(at 227.33 120.65 180)
 		(fields_autoplaced yes)
 		(effects
@@
 	)
 	(label "Z2_FI4.LHC_CLK_HQ_N"
-		(at 227.33 77.47 180)
+		(at 227.33 74.93 180)
 		(fields_autoplaced yes)
 		(effects
@@
 	)
 	(label "Z2_FI3.LHC_CLK_HQ_N"
-		(at 227.33 69.85 180)
+		(at 227.33 67.31 180)
 		(fields_autoplaced yes)
 		(effects
@@
 	)
 	(label "Z2_FI5.LHC_CLK_HQ_N"
-		(at 227.33 85.09 180)
+		(at 227.33 82.55 180)
 		(fields_autoplaced yes)
 		(effects
@@
 	)
 	(label "Z2_FI4.LHC_CLK_HQ_P"
-		(at 227.33 74.93 180)
+		(at 227.33 77.47 180)
 		(fields_autoplaced yes)
 		(effects
@@
 	)
 	(label "Z2_FI2.LHC_CLK_HQ_N"
+		(at 227.33 59.69 180)
+		(fields_autoplaced yes)
+		(effects
+			(font
+				(size 1.27 1.27)
+			)
+			(justify right bottom)
+		)
+	)
+	(label "Z2_FI9.LHC_CLK_HQ_N"
+		(at 227.33 113.03 180)
+		(fields_autoplaced yes)
+		(effects
+			(font
+				(size 1.27 1.27)
+			)
+			(justify right bottom)
+		)
+	)
+	(label "Z2_FI6.LHC_CLK_HQ_P"
+		(at 227.33 92.71 180)
+		(fields_autoplaced yes)
+		(effects
+			(font
+				(size 1.27 1.27)
+			)
+			(justify right bottom)
+		)
+	)
+	(label "Z2_FI7.LHC_CLK_HQ_N"
+		(at 227.33 97.79 180)
+		(fields_autoplaced yes)
+		(effects
+			(font
+				(size 1.27 1.27)
+			)
+			(justify right bottom)
+		)
+	)
+	(label "Z2_FI2.LHC_CLK_HQ_P"
 		(at 227.33 62.23 180)
 		(fields_autoplaced yes)
@@
 		)
 	)
-	(label "Z2_FI9.LHC_CLK_HQ_N"
-		(at 227.33 115.57 180)
-		(fields_autoplaced yes)
-		(effects
-			(font
-				(size 1.27 1.27)
-			)
-			(justify right bottom)
-		)
-	)
-	(label "Z2_FI6.LHC_CLK_HQ_P"
-		(at 227.33 90.17 180)
-		(fields_autoplaced yes)
-		(effects
-			(font
-				(size 1.27 1.27)
-			)
-			(justify right bottom)
-		)
-	)
-	(label "Z2_FI7.LHC_CLK_HQ_N"
-		(at 227.33 100.33 180)
-		(fields_autoplaced yes)
-		(effects
-			(font
-				(size 1.27 1.27)
-			)
-			(justify right bottom)
-		)
-	)
-	(label "Z2_FI2.LHC_CLK_HQ_P"
-		(at 227.33 59.69 180)
-		(fields_autoplaced yes)
-		(effects
-			(font
-				(size 1.27 1.27)
-			)
-			(justify right bottom)
-		)
-	)
 	(label "Z2_FI8.LHC_CLK_HQ_N"
+		(at 227.33 105.41 180)
+		(fields_autoplaced yes)
+		(effects
+			(font
+				(size 1.27 1.27)
+			)
+			(justify right bottom)
+		)
+	)
+	(label "Z2_FI8.LHC_CLK_HQ_P"
 		(at 227.33 107.95 180)
 		(fields_autoplaced yes)
 		(effects
-			(font
-				(size 1.27 1.27)
-			)
-			(justify right bottom)
-		)
-	)
-	(label "Z2_FI8.LHC_CLK_HQ_P"
-		(at 227.33 105.41 180)
-		(fields_autoplaced yes)
-		(effects
